Commit message: working forward kinematics demo

File: unity_ros_backend/unity_robot_description/urdf/ur5e_2f_85.urdf (robot description, URDF)
Before this commit: robot ur5e_2f_85_gripper, 22 links, 21 joints
Links:
- link base_link_inertia: geometry collision mesh filename=package://ur_description/meshes/ur5e/collision/base.stl; visual mesh filename=package://ur_description/meshes/ur5e/visual/base.dae
- link forearm_link: geometry collision mesh filename=package://ur_description/meshes/ur5e/collision/forearm.stl; visual mesh filename=package://ur_description/meshes/ur5e/visual/forearm.dae
- link left_inner_finger: geometry collision mesh filename=package://robotiq_2f_85_gripper_visualization/meshes/collis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 scale=0.001 0.001 0.001; visual mesh filename=package://robotiq_2f_85_gripper_visualization/meshes/visual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 scale=0.001 0.001 0.001
- link left_inner_knuckle: geometry collision mesh filename=package://robotiq_2f_85_gripper_visualization/meshes/collis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 scale=0.001 0.001 0.001; visual mesh filename=package://robotiq_2f_85_gripper_visualization/meshes/visual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 scale=0.001 0.001 0.001
- link left_outer_finger: geometry collision mesh filename=package://robotiq_2f_85_gripper_visualization/meshes/collis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 scale=0.001 0.001 0.001; visual mesh filename=package://robotiq_2f_85_gripper_visualization/meshes/visual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 scale=0.001 0.001 0.001
- link left_outer_knuckle: geometry collision mesh filename=package://robotiq_2f_85_gripper_visualization/meshes/collis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 scale=0.001 0.001 0.001; visual mesh filename=package://robotiq_2f_85_gripper_visualization/meshes/visual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 scale=0.001 0.001 0.001
- link right_inner_finger: geometry collision mesh filename=package://robotiq_2f_85_gripper_visualization/meshes/collis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 scale=0.001 0.001 0.001; visual mesh filename=package://robotiq_2f_85_gripper_visualization/meshes/visual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 scale=0.001 0.001 0.001
- link right_inner_knuckle: geometry collision mesh filename=package://robotiq_2f_85_gripper_visualization/meshes/collis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 scale=0.001 0.001 0.001; visual mesh filename=package://robotiq_2f_85_gripper_visualization/meshes/visual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 scale=0.001 0.001 0.001
- link right_outer_finger: geometry collision mesh filename=package://robotiq_2f_85_gripper_visualization/meshes/collis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 scale=0.001 0.001 0.001; visual mesh filename=package://robotiq_2f_85_gripper_visualization/meshes/visual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 scale=0.001 0.001 0.001
- link right_outer_knuckle: geometry collision mesh filename=package://robotiq_2f_85_gripper_visualization/meshes/collis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 scale=0.001 0.001 0.001; visual mesh filename=package://robotiq_2f_85_gripper_visualization/meshes/visual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 scale=0.001 0.001 0.001
- link robotiq_arg2f_base_link: geometry collision mesh filename=package://robotiq_2f_85_gripper_visualization/meshes/collis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; visual mesh filename=package://robotiq_2f_85_gripper_visualization/meshes/visual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
- link shoulder_link: geometry collision mesh filename=package://ur_description/meshes/ur5e/collision/shoulder.stl; visual mesh filename=package://ur_description/meshes/ur5e/visual/shoulder.dae
- link upper_arm_link: geometry collision mesh filename=package://ur_description/meshes/ur5e/collision/upperarm.stl; visual mesh filename=package://ur_description/meshes/ur5e/visual/upperarm.dae
- link wrist_1_link: geometry collision mesh filename=package://ur_description/meshes/ur5e/collision/wrist1.stl; visual mesh filename=package://ur_description/meshes/ur5e/visual/wrist1.dae
- link wrist_2_link: geometry collision mesh filename=package://ur_description/meshes/ur5e/collision/wrist2.stl; visual mesh filename=package://ur_description/meshes/ur5e/visual/wrist2.dae
- link wrist_3_link: geometry collision mesh filename=package://ur_description/meshes/ur5e/collision/wrist3.stl; visual mesh filename=package://ur_description/meshes/ur5e/visual/wrist3.dae
Joints:
- removed joint tool0-gripper_base
- added joint ur5e_tool0-gripper_base: type fixed, parent tool0, child robotiq_arg2f_base_link, origin xyz=0.0 0.0 0.0 rpy=0.0 0.0 0.0
