Commit message: remove Unity package and updated robot description files

File: unity_ros_backend/unity_robot_description/xacro/macros/robotiq_arg2f_140_macro.xacro (robot description, xacro)
@@ -1,11 +1,11 @@
 <?xml version="1.0"?>
 <robot xmlns:xacro="http://ros.org/wiki/xacro">
-  <xacro:include filename="$(find unity_robot_description)/xacro/macros/robotiq_arg2f_85_transmissions.xacro" />
-  <xacro:macro name="robotiq_arg2f_85" params="
+  <xacro:include filename="$(find unity_robot_description)/xacro/macros/robotiq_arg2f_140_transmissions.xacro" />
+  <xacro:macro name="robotiq_arg2f_140" params="
     prefix
     transmission_hw_interface:=hardware/interface/EffortJointInterface"
   >
     <!-- Add URDF transmission elements (for ros_control) -->
-    <xacro:robotiq_arg2f_85_transmission prefix="${prefix}" hw_interface="${transmission_hw_interface}"/>
+    <xacro:robotiq_arg2f_140_transmission prefix="${prefix}" hw_interface="${transmission_hw_interface}"/>
     <!-- fingers links macros -->
     <xacro:macro name="outer_knuckle" params="prefix fingerprefix">
@@ -19,5 +19,5 @@
           <origin xyz="0 0 0" rpy="0 0 0" />
           <geometry>
-            <mesh filename="package://unity_robot_description/models/robotiq_2f_85/visual/robotiq_arg2f_85_outer_knuckle.dae" scale="0.001 0.001 0.001"/>
+            <mesh filename="package://unity_robot_description/models/robotiq_2f_140/visual/robotiq_arg2f_140_outer_knuckle.stl"/>
           </geometry>
           <material name="">
@@ -28,5 +28,5 @@
           <origin xyz="0 0 0" rpy="0 0 0" />
           <geometry>
-            <mesh filename="package://unity_robot_description/models/robotiq_2f_85/collision/robotiq_arg2f_85_outer_knuckle.dae" scale="0.001 0.001 0.001"/>
+            <mesh filename="package://unity_robot_description/models/robotiq_2f_140/collision/robotiq_arg2f_140_outer_knuckle.stl"/>
           </geometry>
         </collision>
@@ -43,14 +43,14 @@
           <origin xyz="0 0 0" rpy="0 0 0" />
           <geometry>
-            <mesh filename="package://unity_robot_description/models/robotiq_2f_85/visual/robotiq_arg2f_85_outer_finger.dae" scale="0.001 0.001 0.001"/>
-          </geometry>
-          <material name="">
-            <color rgba="0.1 0.1 0.1 1" />
-          </material>
-        </visual>
-        <collision>
-          <origin xyz="0 0 0" rpy="0 0 0" />
-          <geometry>
-            <mesh filename="package://unity_robot_description/models/robotiq_2f_85/collision/robotiq_arg2f_85_outer_finger.dae" scale="0.001 0.001 0.001"/>
+            <mesh filename="package://unity_robot_description/models/robotiq_2f_140/visual/robotiq_arg2f_140_outer_finger.stl"/>
+          </geometry>
+          <material name="">
+            <color rgba="0.1 0.1 0.1 1" />
+          </material>
+        </visual>
+        <collision>
+          <origin xyz="0 0 0" rpy="0 0 0" />
+          <geometry>
+            <mesh filename="package://unity_robot_description/models/robotiq_2f_140/collision/robotiq_arg2f_140_outer_finger.stl"/>
           </geometry>
         </collision>
@@ -67,14 +67,14 @@
           <origin xyz="0 0 0" rpy="0 0 0" />
           <geometry>
-            <mesh filename="package://unity_robot_description/models/robotiq_2f_85/visual/robotiq_arg2f_85_inner_knuckle.dae" scale="0.001 0.001 0.001"/>
-          </geometry>
-          <material name="">
-            <color rgba="0.1 0.1 0.1 1" />
-          </material>
-        </visual>
-        <collision>
-          <origin xyz="0 0 0" rpy="0 0 0" />
-          <geometry>
-            <mesh filename="package://unity_robot_description/models/robotiq_2f_85/collision/robotiq_arg2f_85_inner_knuckle.dae" scale="0.001 0.001 0.001"/>
+            <mesh filename="package://unity_robot_description/models/robotiq_2f_140/visual/robotiq_arg2f_140_inner_knuckle.stl"/>
+          </geometry>
+          <material name="">
+            <color rgba="0.1 0.1 0.1 1" />
+          </material>
+        </visual>
+        <collision>
+          <origin xyz="0 0 0" rpy="0 0 0" />
+          <geometry>
+            <mesh filename="package://unity_robot_description/models/robotiq_2f_140/collision/robotiq_arg2f_140_inner_knuckle.stl"/>
           </geometry>
         </collision>
@@ -91,14 +91,14 @@
           <origin xyz="0 0 0" rpy="0 0 0" />
           <geometry>
-            <mesh filename="package://unity_robot_description/models/robotiq_2f_85/visual/robotiq_arg2f_85_inner_finger.dae" scale="0.001 0.001 0.001"/>
-          </geometry>
-          <material name="">
-            <color rgba="0.1 0.1 0.1 1" />
-          </material>
-        </visual>
-        <collision>
-          <origin xyz="0 0 0" rpy="0 0 0" />
-          <geometry>
-            <mesh filename="package://unity_robot_description/models/robotiq_2f_85/collision/robotiq_arg2f_85_inner_finger.dae" scale="0.001 0.001 0.001" />
+            <mesh filename="package://unity_robot_description/models/robotiq_2f_140/visual/robotiq_arg2f_140_inner_finger.stl"/>
+          </geometry>
+          <material name="">
+            <color rgba="0.1 0.1 0.1 1" />
+          </material>
+        </visual>
+        <collision>
+          <origin xyz="0 0 0" rpy="0 0 0" />
+          <geometry>
+            <mesh filename="package://unity_robot_description/models/robotiq_2f_140/collision/robotiq_arg2f_140_inner_finger.stl" />
           </geometry>
         </collision>
@@ -107,25 +107,25 @@
     <!-- Finger pad link, the default are the "big pads" with rubber-->
     <xacro:macro name="inner_finger_pad" params="prefix fingerprefix">
-      <link name="${prefix}${fingerprefix}_inner_finger_pad">
-        <visual>
-          <origin xyz="0 0 0" rpy="0 0 0" />
-          <geometry>
-            <box size="0.022 0.00635 0.0375"/>
-          </geometry>
-          <material name="">
-            <color rgba="0.9 0.9 0.9 1" />
-          </material>
-        </visual>
-        <collision>
-          <origin xyz="0 0 0" rpy="0 0 0" />
-          <geometry>
-            <box size="0.022 0.00635 0.0375"/>
-          </geometry>
-          <material name="">
-            <color rgba="0.9 0.0 0.0 1" />
-          </material>
-        </collision>
-      </link>
-    </xacro:macro>
+    <link name="${prefix}${fingerprefix}_inner_finger_pad">
+      <visual>
+        <origin xyz="0 0 0" rpy="0 0 0" />
+        <geometry>
+          <box size="0.027 0.065 0.0075"/>
+        </geometry>
+        <material name="">
+          <color rgba="0.9 0.9 0.9 1" />
+        </material>
+      </visual>
+      <collision>
+        <origin xyz="0 0 0" rpy="0 0 0" />
+        <geometry>
+           <box size="0.03 0.07 0.0075"/>
+        </geometry>
+        <material name="">
+          <color rgba="0.9 0.0 0.0 1" />
+        </material>
+      </collision>
+    </link>
+  </xacro:macro>
     <xacro:macro name="finger_links" params="prefix fingerprefix">
       <xacro:outer_knuckle prefix="${prefix}" fingerprefix="${fingerprefix}"/>
@@ -138,5 +138,5 @@
     <xacro:macro name="outer_finger_joint" params="prefix fingerprefix">
       <joint name="${prefix}${fingerprefix}_outer_finger_joint" type="fixed">
-        <origin xyz="0 0.0315 -0.0041" rpy="0 0 0"/>
+        <origin xyz="0 0.01821998610742 0.0260018192872234" rpy="0 0 0" />
         <parent link="${prefix}${fingerprefix}_outer_knuckle" />
         <child link="${prefix}${fingerprefix}_outer_finger" />
@@ -146,26 +146,25 @@
     <xacro:macro name="inner_knuckle_joint" params="prefix fingerprefix reflect">
       <joint name="${prefix}${fingerprefix}_inner_knuckle_joint" type="revolute">
-        <!-- <origin xyz="0 ${reflect * -0.0127} 0.06142" rpy="${pi / 2 + .725} 0 ${(reflect - 1) * pi / 2}" /> -->
-        <origin xyz="0 ${reflect * -0.0127} 0.06142" rpy="0 0 ${(1 + reflect) * pi / 2}"/>
+        <origin xyz="0 ${reflect * -0.0127} 0.06142" rpy="${pi / 2 + .725} 0 ${(reflect - 1) * pi / 2}" />
         <parent link="${prefix}robotiq_arg2f_base_link" />
         <child link="${prefix}${fingerprefix}_inner_knuckle" />
         <axis xyz="1 0 0" />
-        <limit lower="0" upper="0.8757" velocity="0.5" effort="1000" />
-        <mimic joint="${prefix}finger_joint" multiplier="1" offset="0" />
+        <limit lower="-0.8757" upper="0" velocity="0.5" effort="1000" />
+        <mimic joint="${prefix}finger_joint" multiplier="-1" offset="0" />
       </joint>
     </xacro:macro>
     <xacro:macro name="inner_finger_joint" params="prefix fingerprefix">
       <joint name="${prefix}${fingerprefix}_inner_finger_joint" type="revolute">
-        <origin xyz="0 0.0061 0.0471" rpy="0 0 0"/>
+        <origin xyz="0 0.0817554015893473 -0.0282203446692936" rpy="-0.725 0 0" />
         <parent link="${prefix}${fingerprefix}_outer_finger" />
         <child link="${prefix}${fingerprefix}_inner_finger" />
         <axis xyz="1 0 0" />
-        <limit lower="-0.8757" upper="0" velocity="0.5" effort="1000" />
-        <mimic joint="${prefix}finger_joint" multiplier="-1" offset="0" />
+        <limit lower="0" upper="0.8757" velocity="0.5" effort="1000" />
+        <mimic joint="${prefix}finger_joint" multiplier="1" offset="0" />
       </joint>
     </xacro:macro>
     <xacro:macro name="inner_finger_pad_joint" params="prefix fingerprefix">
       <joint name="${prefix}${fingerprefix}_inner_finger_pad_joint" type="fixed">
-        <origin xyz="0 -0.0220203446692936 0.03242" rpy="0 0 0"/>
+        <origin xyz="0 0.0457554015893473 -0.0272203446692936" rpy="0 0 0" />
         <parent link="${prefix}${fingerprefix}_inner_finger" />
         <child link="${prefix}${fingerprefix}_inner_finger_pad" />
@@ -195,14 +194,14 @@
           <origin xyz="0 0 0" rpy="0 0 0" />
           <geometry>
-            <mesh filename="package://unity_robot_description/models/robotiq_2f_85/visual/robotiq_arg2f_base_link.stl" />
-          </geometry>
-          <material name="">
-            <color rgba="0.1 0.1 0.1 1" />
-          </material>
-        </visual>
-        <collision>
-          <origin xyz="0 0 0" rpy="0 0 0" />
-          <geometry>
-            <mesh filename="package://unity_robot_description/models/robotiq_2f_85/collision/robotiq_arg2f_base_link.stl" />
+            <mesh filename="package://unity_robot_description/models/robotiq_2f_140/visual/robotiq_arg2f_base_link.stl" />
+          </geometry>
+          <material name="">
+            <color rgba="0.1 0.1 0.1 1" />
+          </material>
+        </visual>
+        <collision>
+          <origin xyz="0 0 0" rpy="0 0 0" />
+          <geometry>
+            <mesh filename="package://unity_robot_description/models/robotiq_2f_140/collision/robotiq_arg2f_base_link.stl" />
           </geometry>
         </collision>
@@ -212,9 +211,9 @@
     <xacro:finger_joints prefix="${prefix}" fingerprefix="left" reflect="1.0"/>
     <joint name="${prefix}finger_joint" type="revolute">
-      <origin xyz="0 -0.0306011 0.054904" rpy="0 0 ${pi}"/>
+      <origin xyz="0 -0.0306011 0.054904" rpy="${pi / 2 + .725} 0 0"/>
       <parent link="${prefix}robotiq_arg2f_base_link" />
       <child link="${prefix}left_outer_knuckle" />
-      <axis xyz="1 0 0" />
-      <limit lower="0" upper="0.8" velocity="0.5" effort="1000" />
+      <axis xyz="-1 0 0" />
+      <limit lower="0" upper="0.7" velocity="0.5" effort="1000" />
     </joint>
     <!-- right finger -->
@@ -222,10 +221,10 @@
     <xacro:finger_links prefix="${prefix}" fingerprefix="right"/>
     <joint name="${prefix}right_finger_joint" type="revolute">
-      <origin xyz="0 0.0306011 0.054904" rpy="0 0 0"/>
+      <origin xyz="0 0.0306011 0.054904" rpy="${pi / 2 + .725} 0 ${pi}"/>
       <parent link="${prefix}robotiq_arg2f_base_link" />
       <child link="${prefix}right_outer_knuckle" />
       <axis xyz="1 0 0" />
-      <limit lower="0" upper="0.81" velocity="0.5" effort="1000" />
-      <mimic joint="${prefix}finger_joint" multiplier="1" offset="0" />
+      <limit lower="-0.725" upper="0" velocity="0.5" effort="1000" />
+      <mimic joint="${prefix}finger_joint" multiplier="-1" offset="0" />
     </joint>
   </xacro:macro>
