Commit message: updated MoveIt! planning to include center point of extended gripper

File: unity_ros_backend/unity_robot_description/xacro/macros/robotiq_arg2f_85_macro.xacro (robot description, xacro)
@@ -207,5 +207,5 @@
           </geometry>
         </collision>
-      </link>
+    </link>
     <!-- left finger -->
     <xacro:finger_links prefix="${prefix}" fingerprefix="left"/>
