Commit message: modified xacro and MoveIt! to plan with fixed open gripper

File: catkin_ws/src/unity_ros_backend/unity_robot_description/urdf/ur5e_robotiq_2f_85.urdf (robot description, URDF)
Before this commit: robot ur5e_robotiq_85_gripper, 23 links, 22 joints
Links:
- link left_inner_finger_pad: mass 0.1 -> None
- link right_inner_finger_pad: mass 0.1 -> None
Joints:
- joint finger_joint: type revolute -> fixed
- joint left_inner_finger_joint: type revolute -> fixed
- joint left_inner_knuckle_joint: type revolute -> fixed
- joint right_finger_joint: type revolute -> fixed
- joint right_inner_finger_joint: type revolute -> fixed
- joint right_inner_knuckle_joint: type revolute -> fixed

File: catkin_ws/src/unity_ros_backend/unity_robot_description/xacro/macros/robotiq_arg2f_85_macro_fixed.xacro (robot description, xacro)
@@ -145,5 +145,5 @@
     </xacro:macro>
     <xacro:macro name="inner_knuckle_joint" params="prefix fingerprefix reflect">
-      <joint name="${prefix}${fingerprefix}_inner_knuckle_joint" type="revolute">
+      <joint name="${prefix}${fingerprefix}_inner_knuckle_joint" type="fixed">
         <!-- <origin xyz="0 ${reflect * -0.0127} 0.06142" rpy="${pi / 2 + .725} 0 ${(reflect - 1) * pi / 2}" /> -->
         <origin xyz="0 ${reflect * -0.0127} 0.06142" rpy="0 0 ${(1 + reflect) * pi / 2}"/>
@@ -156,5 +156,5 @@
     </xacro:macro>
     <xacro:macro name="inner_finger_joint" params="prefix fingerprefix">
-      <joint name="${prefix}${fingerprefix}_inner_finger_joint" type="revolute">
+      <joint name="${prefix}${fingerprefix}_inner_finger_joint" type="fixed">
         <origin xyz="0 0.0061 0.0471" rpy="0 0 0"/>
         <parent link="${prefix}${fingerprefix}_outer_finger" />
@@ -211,5 +211,5 @@
     <xacro:finger_links prefix="${prefix}" fingerprefix="left"/>
     <xacro:finger_joints prefix="${prefix}" fingerprefix="left" reflect="1.0"/>
-    <joint name="${prefix}finger_joint" type="revolute">
+    <joint name="${prefix}finger_joint" type="fixed">
       <origin xyz="0 -0.0306011 0.054904" rpy="0 0 ${pi}"/>
       <parent link="${prefix}robotiq_arg2f_base_link" />
@@ -221,5 +221,5 @@
     <xacro:finger_links prefix="${prefix}" fingerprefix="right"/>
     <xacro:finger_joints prefix="${prefix}" fingerprefix="right" reflect="-1.0"/>
-    <joint name="${prefix}right_finger_joint" type="revolute">
+    <joint name="${prefix}right_finger_joint" type="fixed">
       <origin xyz="0 0.0306011 0.054904" rpy="0 0 0"/>
       <parent link="${prefix}robotiq_arg2f_base_link" />

File: catkin_ws/src/unity_ros_backend/unity_robot_description/xacro/ur5e_robotiq_2f_85.xacro (robot description, xacro)
@@ -2,5 +2,5 @@
 <robot xmlns:xacro="http://www.ros.org/wiki/xacro" name="ur5e_robotiq_85_gripper">
     <xacro:include filename="$(find unity_robot_description)/xacro/macros/ur5e_macro.xacro" />
-    <xacro:include filename="$(find unity_robot_description)/xacro/macros/robotiq_arg2f_85_macro.xacro" />
+    <xacro:include filename="$(find unity_robot_description)/xacro/macros/robotiq_arg2f_85_macro_fixed.xacro" />
     <xacro:property name="coupling_offset" value="0.0" />
     <xacro:property name="gripper_height" value="0.1628" />
