Commit message: moveit tracking of gripper position

File: catkin_ws/src/unity_ros_backend/unity_robot_description/urdf/ur5e_robotiq_2f_85_fixed.urdf (robot description, URDF)
Before this commit: robot ur5e_robotiq_85_gripper, 23 links, 22 joints
Joints:
- joint finger_joint: type revolute -> fixed
- joint left_inner_finger_joint: type revolute -> fixed
- joint left_inner_knuckle_joint: type revolute -> fixed
- joint right_finger_joint: type revolute -> fixed
- joint right_inner_finger_joint: type revolute -> fixed
- joint right_inner_knuckle_joint: type revolute -> fixed
