Commit message: updated MoveIt! planning to include L515 and plate

File: catkin_ws/src/unity_ros_backend/unity_robot_description/xacro/macros/robotiq-3f-gripper_articulated_macro.xacro (robot description, xacro)
@@ -15,5 +15,5 @@
 			<visual>
 				<geometry>
-					<mesh filename="package://unity_robot_description/models/robotiq_3f_articulated/visual/palm.dae" />
+					<mesh filename="package://unity_robot_description/models/robotiq/robotiq_3f_articulated/visual/palm.dae" />
 				</geometry>
 				<material name="gray">
@@ -23,5 +23,5 @@
 			<collision>
 				<geometry>
-					<mesh filename="package://unity_robot_description/models/robotiq_3f_articulated/collision/palm.STL" />
+					<mesh filename="package://unity_robot_description/models/robotiq/robotiq_3f_articulated/collision/palm.STL" />
 				</geometry>
 				<material name="yellow">

File: catkin_ws/src/unity_ros_backend/unity_robot_description/xacro/macros/robotiq-3f-gripper_finger_articulated_macro.xacro (robot description, xacro)
@@ -12,5 +12,5 @@
 				<origin xyz="0.020 0 0" rpy="0 0 0"/>
 				<geometry>
-					<mesh filename="package://unity_robot_description/models/robotiq_3f_articulated/visual/link_0.dae" />
+					<mesh filename="package://unity_robot_description/models/robotiq/robotiq_3f_articulated/visual/link_0.dae" />
 				</geometry>
 				<material name="gray">
@@ -21,5 +21,5 @@
 				<origin xyz="0.020 0 0" rpy="0 0 0"/>
 				<geometry>
-					<mesh filename="package://unity_robot_description/models/robotiq_3f_articulated/collision/link_0.STL" />
+					<mesh filename="package://unity_robot_description/models/robotiq/robotiq_3f_articulated/collision/link_0.STL" />
 				</geometry>
 				<material name="yellow">
@@ -37,5 +37,5 @@
 				<origin xyz="0.050 -.028 0" rpy="0 0 -0.52"/>
 				<geometry>
-					<mesh filename="package://unity_robot_description/models/robotiq_3f_articulated/visual/link_1.dae" />
+					<mesh filename="package://unity_robot_description/models/robotiq/robotiq_3f_articulated/visual/link_1.dae" />
 				</geometry>
 				<material name="gray"/>
@@ -44,5 +44,5 @@
 				<origin xyz="0.050 -.028 0" rpy="0 0 -0.52"/>
 				<geometry>
-					<mesh filename="package://unity_robot_description/models/robotiq_3f_articulated/collision/link_1.STL" />
+					<mesh filename="package://unity_robot_description/models/robotiq/robotiq_3f_articulated/collision/link_1.STL" />
 				</geometry>
 				<material name="yellow"/>
@@ -63,5 +63,5 @@
 				<origin xyz="0.039 0 0.0075" rpy="0 0 0"/>
 				<geometry>
-					<mesh filename="package://unity_robot_description/models/robotiq_3f_articulated/visual/link_2.dae" />
+					<mesh filename="package://unity_robot_description/models/robotiq/robotiq_3f_articulated/visual/link_2.dae" />
 				</geometry>
 				<material name="gray"/>
@@ -70,5 +70,5 @@
 				<origin xyz="0.039 0 0.0075" rpy="0 0 0"/>
 				<geometry>
-					<mesh filename="package://unity_robot_description/models/robotiq_3f_articulated/collision/link_2.STL" />
+					<mesh filename="package://unity_robot_description/models/robotiq/robotiq_3f_articulated/collision/link_2.STL" />
 				</geometry>
 				<material name="yellow"/>
@@ -84,5 +84,5 @@
 				<origin xyz="0 0 0" rpy="0 0 0.52"/>
 				<geometry>
-					<mesh filename="package://unity_robot_description/models/robotiq_3f_articulated/visual/link_3.dae" />
+					<mesh filename="package://unity_robot_description/models/robotiq/robotiq_3f_articulated/visual/link_3.dae" />
 				</geometry>
 				<material name="gray"/>
@@ -91,5 +91,5 @@
 				<origin xyz="0 0 0" rpy="0 0 0.52"/>
 				<geometry>
-					<mesh filename="package://unity_robot_description/models/robotiq_3f_articulated/collision/link_3.STL" />
+					<mesh filename="package://unity_robot_description/models/robotiq/robotiq_3f_articulated/collision/link_3.STL" />
 				</geometry>
 				<material name="yellow"/>

File: catkin_ws/src/unity_ros_backend/unity_robot_description/xacro/macros/robotiq-3f-gripper_mesh_macro.xacro (robot description, xacro)
@@ -5,5 +5,5 @@
 			<visual>
 				<geometry>
-                	<mesh filename="package://unity_robot_description/models/robotiq_3f/visual/GRIPPER_OPEN_PALM.stl" />
+                	<mesh filename="package://unity_robot_description/models/robotiq/robotiq_3f/visual/GRIPPER_OPEN_PALM.stl" />
 				</geometry>
 				<material name="green">
@@ -13,5 +13,5 @@
 			<collision>
 				<geometry>
-                	<mesh filename="package://unity_robot_description/models/robotiq_3f/collision/GRIPPER_OPEN_PALM.stl" />
+                	<mesh filename="package://unity_robot_description/models/robotiq/robotiq_3f/collision/GRIPPER_OPEN_PALM.stl" />
 				</geometry>
 				<material name="yellow">
@@ -23,5 +23,5 @@
 			<visual>
 				<geometry>
-                	<mesh filename="package://unity_robot_description/models/robotiq_3f/visual/GRIPPER_OPEN_FINGER_1.stl" />
+                	<mesh filename="package://unity_robot_description/models/robotiq/robotiq_3f/visual/GRIPPER_OPEN_FINGER_1.stl" />
 				</geometry>
 				<material name="green"/>
@@ -29,5 +29,5 @@
 			<collision>
 				<geometry>
-                	<mesh filename="package://unity_robot_description/models/robotiq_3f/collision/GRIPPER_OPEN_FINGER_1.stl" />
+                	<mesh filename="package://unity_robot_description/models/robotiq/robotiq_3f/collision/GRIPPER_OPEN_FINGER_1.stl" />
 				</geometry>
 				<material name="yellow"/>
@@ -37,5 +37,5 @@
 			<visual>
 				<geometry>
-                	<mesh filename="package://unity_robot_description/models/robotiq_3f/visual/GRIPPER_OPEN_FINGER_2.stl" />
+                	<mesh filename="package://unity_robot_description/models/robotiq/robotiq_3f/visual/GRIPPER_OPEN_FINGER_2.stl" />
 				</geometry>
 				<material name="green"/>
@@ -43,5 +43,5 @@
 			<collision>
 				<geometry>
-                	<mesh filename="package://unity_robot_description/models/robotiq_3f/collision/GRIPPER_OPEN_FINGER_2.stl" />
+                	<mesh filename="package://unity_robot_description/models/robotiq/robotiq_3f/collision/GRIPPER_OPEN_FINGER_2.stl" />
 				</geometry>
 				<material name="yellow"/>
@@ -51,5 +51,5 @@
 			<visual>
 				<geometry>
-                	<mesh filename="package://unity_robot_description/models/robotiq_3f/visual/GRIPPER_OPEN_FINGER_3.stl" />
+                	<mesh filename="package://unity_robot_description/models/robotiq/robotiq_3f/visual/GRIPPER_OPEN_FINGER_3.stl" />
 				</geometry>
 				<material name="green"/>
@@ -57,5 +57,5 @@
 			<collision>
 				<geometry>
-                	<mesh filename="package://unity_robot_description/models/robotiq_3f/collision/GRIPPER_OPEN_FINGER_3.stl" />
+                	<mesh filename="package://unity_robot_description/models/robotiq/robotiq_3f/collision/GRIPPER_OPEN_FINGER_3.stl" />
 				</geometry>
 				<material name="yellow"/>

File: catkin_ws/src/unity_ros_backend/unity_robot_description/xacro/macros/robotiq_arg2f_140_macro.xacro (robot description, xacro)
@@ -19,5 +19,5 @@
           <origin xyz="0 0 0" rpy="0 0 0" />
           <geometry>
-            <mesh filename="package://unity_robot_description/models/robotiq_2f_140/visual/robotiq_arg2f_140_outer_knuckle.stl"/>
+            <mesh filename="package://unity_robot_description/models/robotiq/robotiq_2f_140/visual/robotiq_arg2f_140_outer_knuckle.stl"/>
           </geometry>
           <material name="">
@@ -28,5 +28,5 @@
           <origin xyz="0 0 0" rpy="0 0 0" />
           <geometry>
-            <mesh filename="package://unity_robot_description/models/robotiq_2f_140/collision/robotiq_arg2f_140_outer_knuckle.stl"/>
+            <mesh filename="package://unity_robot_description/models/robotiq/robotiq_2f_140/collision/robotiq_arg2f_140_outer_knuckle.stl"/>
           </geometry>
         </collision>
@@ -43,14 +43,14 @@
           <origin xyz="0 0 0" rpy="0 0 0" />
           <geometry>
-            <mesh filename="package://unity_robot_description/models/robotiq_2f_140/visual/robotiq_arg2f_140_outer_finger.stl"/>
-          </geometry>
-          <material name="">
-            <color rgba="0.1 0.1 0.1 1" />
-          </material>
-        </visual>
-        <collision>
-          <origin xyz="0 0 0" rpy="0 0 0" />
-          <geometry>
-            <mesh filename="package://unity_robot_description/models/robotiq_2f_140/collision/robotiq_arg2f_140_outer_finger.stl"/>
+            <mesh filename="package://unity_robot_description/models/robotiq/robotiq_2f_140/visual/robotiq_arg2f_140_outer_finger.stl"/>
+          </geometry>
+          <material name="">
+            <color rgba="0.1 0.1 0.1 1" />
+          </material>
+        </visual>
+        <collision>
+          <origin xyz="0 0 0" rpy="0 0 0" />
+          <geometry>
+            <mesh filename="package://unity_robot_description/models/robotiq/robotiq_2f_140/collision/robotiq_arg2f_140_outer_finger.stl"/>
           </geometry>
         </collision>
@@ -67,14 +67,14 @@
           <origin xyz="0 0 0" rpy="0 0 0" />
           <geometry>
-            <mesh filename="package://unity_robot_description/models/robotiq_2f_140/visual/robotiq_arg2f_140_inner_knuckle.stl"/>
-          </geometry>
-          <material name="">
-            <color rgba="0.1 0.1 0.1 1" />
-          </material>
-        </visual>
-        <collision>
-          <origin xyz="0 0 0" rpy="0 0 0" />
-          <geometry>
-            <mesh filename="package://unity_robot_description/models/robotiq_2f_140/collision/robotiq_arg2f_140_inner_knuckle.stl"/>
+            <mesh filename="package://unity_robot_description/models/robotiq/robotiq_2f_140/visual/robotiq_arg2f_140_inner_knuckle.stl"/>
+          </geometry>
+          <material name="">
+            <color rgba="0.1 0.1 0.1 1" />
+          </material>
+        </visual>
+        <collision>
+          <origin xyz="0 0 0" rpy="0 0 0" />
+          <geometry>
+            <mesh filename="package://unity_robot_description/models/robotiq/robotiq_2f_140/collision/robotiq_arg2f_140_inner_knuckle.stl"/>
           </geometry>
         </collision>
@@ -91,14 +91,14 @@
           <origin xyz="0 0 0" rpy="0 0 0" />
           <geometry>
-            <mesh filename="package://unity_robot_description/models/robotiq_2f_140/visual/robotiq_arg2f_140_inner_finger.stl"/>
-          </geometry>
-          <material name="">
-            <color rgba="0.1 0.1 0.1 1" />
-          </material>
-        </visual>
-        <collision>
-          <origin xyz="0 0 0" rpy="0 0 0" />
-          <geometry>
-            <mesh filename="package://unity_robot_description/models/robotiq_2f_140/collision/robotiq_arg2f_140_inner_finger.stl" />
+            <mesh filename="package://unity_robot_description/models/robotiq/robotiq_2f_140/visual/robotiq_arg2f_140_inner_finger.stl"/>
+          </geometry>
+          <material name="">
+            <color rgba="0.1 0.1 0.1 1" />
+          </material>
+        </visual>
+        <collision>
+          <origin xyz="0 0 0" rpy="0 0 0" />
+          <geometry>
+            <mesh filename="package://unity_robot_description/models/robotiq/robotiq_2f_140/collision/robotiq_arg2f_140_inner_finger.stl" />
           </geometry>
         </collision>
@@ -194,14 +194,14 @@
           <origin xyz="0 0 0" rpy="0 0 0" />
           <geometry>
-            <mesh filename="package://unity_robot_description/models/robotiq_2f_140/visual/robotiq_arg2f_base_link.stl" />
-          </geometry>
-          <material name="">
-            <color rgba="0.1 0.1 0.1 1" />
-          </material>
-        </visual>
-        <collision>
-          <origin xyz="0 0 0" rpy="0 0 0" />
-          <geometry>
-            <mesh filename="package://unity_robot_description/models/robotiq_2f_140/collision/robotiq_arg2f_base_link.stl" />
+            <mesh filename="package://unity_robot_description/models/robotiq/robotiq_2f_140/visual/robotiq_arg2f_base_link.stl" />
+          </geometry>
+          <material name="">
+            <color rgba="0.1 0.1 0.1 1" />
+          </material>
+        </visual>
+        <collision>
+          <origin xyz="0 0 0" rpy="0 0 0" />
+          <geometry>
+            <mesh filename="package://unity_robot_description/models/robotiq/robotiq_2f_140/collision/robotiq_arg2f_base_link.stl" />
           </geometry>
         </collision>

File: catkin_ws/src/unity_ros_backend/unity_robot_description/xacro/macros/robotiq_arg2f_85_macro.xacro (robot description, xacro)
@@ -19,5 +19,5 @@
           <origin xyz="0 0 0" rpy="0 0 0" />
           <geometry>
-            <mesh filename="package://unity_robot_description/models/robotiq_2f_85/visual/robotiq_arg2f_85_outer_knuckle.dae" scale="0.001 0.001 0.001"/>
+            <mesh filename="package://unity_robot_description/models/robotiq/robotiq_2f_85/visual/robotiq_arg2f_85_outer_knuckle.dae" scale="0.001 0.001 0.001"/>
           </geometry>
           <material name="">
@@ -28,5 +28,5 @@
           <origin xyz="0 0 0" rpy="0 0 0" />
           <geometry>
-            <mesh filename="package://unity_robot_description/models/robotiq_2f_85/collision/robotiq_arg2f_85_outer_knuckle.dae" scale="0.001 0.001 0.001"/>
+            <mesh filename="package://unity_robot_description/models/robotiq/robotiq_2f_85/collision/robotiq_arg2f_85_outer_knuckle.dae" scale="0.001 0.001 0.001"/>
           </geometry>
         </collision>
@@ -43,14 +43,14 @@
           <origin xyz="0 0 0" rpy="0 0 0" />
           <geometry>
-            <mesh filename="package://unity_robot_description/models/robotiq_2f_85/visual/robotiq_arg2f_85_outer_finger.dae" scale="0.001 0.001 0.001"/>
-          </geometry>
-          <material name="">
-            <color rgba="0.1 0.1 0.1 1" />
-          </material>
-        </visual>
-        <collision>
-          <origin xyz="0 0 0" rpy="0 0 0" />
-          <geometry>
-            <mesh filename="package://unity_robot_description/models/robotiq_2f_85/collision/robotiq_arg2f_85_outer_finger.dae" scale="0.001 0.001 0.001"/>
+            <mesh filename="package://unity_robot_description/models/robotiq/robotiq_2f_85/visual/robotiq_arg2f_85_outer_finger.dae" scale="0.001 0.001 0.001"/>
+          </geometry>
+          <material name="">
+            <color rgba="0.1 0.1 0.1 1" />
+          </material>
+        </visual>
+        <collision>
+          <origin xyz="0 0 0" rpy="0 0 0" />
+          <geometry>
+            <mesh filename="package://unity_robot_description/models/robotiq/robotiq_2f_85/collision/robotiq_arg2f_85_outer_finger.dae" scale="0.001 0.001 0.001"/>
           </geometry>
         </collision>
@@ -67,14 +67,14 @@
           <origin xyz="0 0 0" rpy="0 0 0" />
           <geometry>
-            <mesh filename="package://unity_robot_description/models/robotiq_2f_85/visual/robotiq_arg2f_85_inner_knuckle.dae" scale="0.001 0.001 0.001"/>
-          </geometry>
-          <material name="">
-            <color rgba="0.1 0.1 0.1 1" />
-          </material>
-        </visual>
-        <collision>
-          <origin xyz="0 0 0" rpy="0 0 0" />
-          <geometry>
-            <mesh filename="package://unity_robot_description/models/robotiq_2f_85/collision/robotiq_arg2f_85_inner_knuckle.dae" scale="0.001 0.001 0.001"/>
+            <mesh filename="package://unity_robot_description/models/robotiq/robotiq_2f_85/visual/robotiq_arg2f_85_inner_knuckle.dae" scale="0.001 0.001 0.001"/>
+          </geometry>
+          <material name="">
+            <color rgba="0.1 0.1 0.1 1" />
+          </material>
+        </visual>
+        <collision>
+          <origin xyz="0 0 0" rpy="0 0 0" />
+          <geometry>
+            <mesh filename="package://unity_robot_description/models/robotiq/robotiq_2f_85/collision/robotiq_arg2f_85_inner_knuckle.dae" scale="0.001 0.001 0.001"/>
           </geometry>
         </collision>
@@ -91,14 +91,14 @@
           <origin xyz="0 0 0" rpy="0 0 0" />
           <geometry>
-            <mesh filename="package://unity_robot_description/models/robotiq_2f_85/visual/robotiq_arg2f_85_inner_finger.dae" scale="0.001 0.001 0.001"/>
-          </geometry>
-          <material name="">
-            <color rgba="0.1 0.1 0.1 1" />
-          </material>
-        </visual>
-        <collision>
-          <origin xyz="0 0 0" rpy="0 0 0" />
-          <geometry>
-            <mesh filename="package://unity_robot_description/models/robotiq_2f_85/collision/robotiq_arg2f_85_inner_finger.dae" scale="0.001 0.001 0.001" />
+            <mesh filename="package://unity_robot_description/models/robotiq/robotiq_2f_85/visual/robotiq_arg2f_85_inner_finger.dae" scale="0.001 0.001 0.001"/>
+          </geometry>
+          <material name="">
+            <color rgba="0.1 0.1 0.1 1" />
+          </material>
+        </visual>
+        <collision>
+          <origin xyz="0 0 0" rpy="0 0 0" />
+          <geometry>
+            <mesh filename="package://unity_robot_description/models/robotiq/robotiq_2f_85/collision/robotiq_arg2f_85_inner_finger.dae" scale="0.001 0.001 0.001" />
           </geometry>
         </collision>
@@ -195,14 +195,14 @@
           <origin xyz="0 0 0" rpy="0 0 0" />
           <geometry>
-            <mesh filename="package://unity_robot_description/models/robotiq_2f_85/visual/robotiq_arg2f_base_link.stl" />
-          </geometry>
-          <material name="">
-            <color rgba="0.1 0.1 0.1 1" />
-          </material>
-        </visual>
-        <collision>
-          <origin xyz="0 0 0" rpy="0 0 0" />
-          <geometry>
-            <mesh filename="package://unity_robot_description/models/robotiq_2f_85/collision/robotiq_arg2f_base_link.stl" />
+            <mesh filename="package://unity_robot_description/models/robotiq/robotiq_2f_85/visual/robotiq_arg2f_base_link.stl" />
+          </geometry>
+          <material name="">
+            <color rgba="0.1 0.1 0.1 1" />
+          </material>
+        </visual>
+        <collision>
+          <origin xyz="0 0 0" rpy="0 0 0" />
+          <geometry>
+            <mesh filename="package://unity_robot_description/models/robotiq/robotiq_2f_85/collision/robotiq_arg2f_base_link.stl" />
           </geometry>
         </collision>
