Commit message: included MoveIt! and Pilz motion planner

File: catkin_ws/src/ur_remote_control/urdf/macros/l515.xacro (robot description, xacro)
@@ -8,6 +8,6 @@
 <robot name="sensor_l515" xmlns:xacro="http://ros.org/wiki/xacro">
   <!-- Includes -->
-  <xacro:include filename="$(find unity_robot_description)/xacro/sensors/realsense/materials.xacro" />
-  <xacro:include filename="$(find unity_robot_description)/xacro/sensors/realsense/usb_plug.xacro" /> <!-- this specific plug does not apply to L515 -->
+  <xacro:include filename="$(find ur_remote_control)/urdf/macros/materials.xacro" />
+  <xacro:include filename="$(find ur_remote_control)/urdf/macros/usb_plug.xacro" /> <!-- this specific plug does not apply to L515 -->
   <xacro:macro name="sensor_l515" params="parent *origin name:=camera use_nominal_extrinsics:=false add_plug:=false use_mesh:=true">
     <xacro:property name="M_PI" value="3.1415926535897931" />
@@ -63,5 +63,5 @@
           <origin xyz="${l515_zero_depth_to_glass} 0 ${-l515_cam_center_to_depth_pz}" rpy="${M_PI/2} 0 ${M_PI/2}"/>
           <geometry>
-              <mesh filename="package://unity_robot_description/models/intel_realsense/l515.dae" />
+              <mesh filename="package://ur_remote_control/models/l515/l515.dae" />
           </geometry>
         </xacro:if>

File: catkin_ws/src/ur_remote_control/urdf/macros/mounting_plate.xacro (robot description, xacro)
@@ -11,5 +11,5 @@
                 <origin xyz="0.0 0.0 0.0" rpy="0.0 0.0 0.0"/>
                 <geometry>
-                    <mesh filename="package://unity_robot_description/models/mounting_plate.stl" />
+                    <mesh filename="package://ur_remote_control/models/mounting_plate.stl" />
                 </geometry>
                 <material name="opague_plastic">

File: catkin_ws/src/ur_remote_control/urdf/macros/robotiq_arg2f_85_macro.xacro (robot description, xacro)
@@ -1,5 +1,5 @@
 <?xml version="1.0"?>
 <robot xmlns:xacro="http://ros.org/wiki/xacro">
-  <xacro:include filename="$(find unity_robot_description)/xacro/macros/robotiq_arg2f_85_transmissions.xacro" />
+  <xacro:include filename="$(find ur_remote_control)/urdf/macros/robotiq_arg2f_85_transmissions.xacro" />
   <xacro:macro name="robotiq_arg2f_85" params="
     prefix
@@ -19,5 +19,5 @@
           <origin xyz="0 0 0" rpy="0 0 0" />
           <geometry>
-            <mesh filename="package://unity_robot_description/models/robotiq/robotiq_2f_85/visual/robotiq_arg2f_85_outer_knuckle.dae" scale="0.001 0.001 0.001"/>
+            <mesh filename="package://ur_remote_control/models/robotiq_2f_85/visual/robotiq_arg2f_85_outer_knuckle.dae" scale="0.001 0.001 0.001"/>
           </geometry>
           <material name="">
@@ -28,5 +28,5 @@
           <origin xyz="0 0 0" rpy="0 0 0" />
           <geometry>
-            <mesh filename="package://unity_robot_description/models/robotiq/robotiq_2f_85/collision/robotiq_arg2f_85_outer_knuckle.dae" scale="0.001 0.001 0.001"/>
+            <mesh filename="package://ur_remote_control/models/robotiq_2f_85/collision/robotiq_arg2f_85_outer_knuckle.dae" scale="0.001 0.001 0.001"/>
           </geometry>
         </collision>
@@ -43,14 +43,14 @@
           <origin xyz="0 0 0" rpy="0 0 0" />
           <geometry>
-            <mesh filename="package://unity_robot_description/models/robotiq/robotiq_2f_85/visual/robotiq_arg2f_85_outer_finger.dae" scale="0.001 0.001 0.001"/>
-          </geometry>
-          <material name="">
-            <color rgba="0.1 0.1 0.1 1" />
-          </material>
-        </visual>
-        <collision>
-          <origin xyz="0 0 0" rpy="0 0 0" />
-          <geometry>
-            <mesh filename="package://unity_robot_description/models/robotiq/robotiq_2f_85/collision/robotiq_arg2f_85_outer_finger.dae" scale="0.001 0.001 0.001"/>
+            <mesh filename="package://ur_remote_control/models/robotiq_2f_85/visual/robotiq_arg2f_85_outer_finger.dae" scale="0.001 0.001 0.001"/>
+          </geometry>
+          <material name="">
+            <color rgba="0.1 0.1 0.1 1" />
+          </material>
+        </visual>
+        <collision>
+          <origin xyz="0 0 0" rpy="0 0 0" />
+          <geometry>
+            <mesh filename="package://ur_remote_control/models/robotiq_2f_85/collision/robotiq_arg2f_85_outer_finger.dae" scale="0.001 0.001 0.001"/>
           </geometry>
         </collision>
@@ -67,14 +67,14 @@
           <origin xyz="0 0 0" rpy="0 0 0" />
           <geometry>
-            <mesh filename="package://unity_robot_description/models/robotiq/robotiq_2f_85/visual/robotiq_arg2f_85_inner_knuckle.dae" scale="0.001 0.001 0.001"/>
-          </geometry>
-          <material name="">
-            <color rgba="0.1 0.1 0.1 1" />
-          </material>
-        </visual>
-        <collision>
-          <origin xyz="0 0 0" rpy="0 0 0" />
-          <geometry>
-            <mesh filename="package://unity_robot_description/models/robotiq/robotiq_2f_85/collision/robotiq_arg2f_85_inner_knuckle.dae" scale="0.001 0.001 0.001"/>
+            <mesh filename="package://ur_remote_control/models/robotiq_2f_85/visual/robotiq_arg2f_85_inner_knuckle.dae" scale="0.001 0.001 0.001"/>
+          </geometry>
+          <material name="">
+            <color rgba="0.1 0.1 0.1 1" />
+          </material>
+        </visual>
+        <collision>
+          <origin xyz="0 0 0" rpy="0 0 0" />
+          <geometry>
+            <mesh filename="package://ur_remote_control/models/robotiq_2f_85/collision/robotiq_arg2f_85_inner_knuckle.dae" scale="0.001 0.001 0.001"/>
           </geometry>
         </collision>
@@ -91,14 +91,14 @@
           <origin xyz="0 0 0" rpy="0 0 0" />
           <geometry>
-            <mesh filename="package://unity_robot_description/models/robotiq/robotiq_2f_85/visual/robotiq_arg2f_85_inner_finger.dae" scale="0.001 0.001 0.001"/>
-          </geometry>
-          <material name="">
-            <color rgba="0.1 0.1 0.1 1" />
-          </material>
-        </visual>
-        <collision>
-          <origin xyz="0 0 0" rpy="0 0 0" />
-          <geometry>
-            <mesh filename="package://unity_robot_description/models/robotiq/robotiq_2f_85/collision/robotiq_arg2f_85_inner_finger.dae" scale="0.001 0.001 0.001" />
+            <mesh filename="package://ur_remote_control/models/robotiq_2f_85/visual/robotiq_arg2f_85_inner_finger.dae" scale="0.001 0.001 0.001"/>
+          </geometry>
+          <material name="">
+            <color rgba="0.1 0.1 0.1 1" />
+          </material>
+        </visual>
+        <collision>
+          <origin xyz="0 0 0" rpy="0 0 0" />
+          <geometry>
+            <mesh filename="package://ur_remote_control/models/robotiq_2f_85/collision/robotiq_arg2f_85_inner_finger.dae" scale="0.001 0.001 0.001" />
           </geometry>
         </collision>
@@ -195,14 +195,14 @@
           <origin xyz="0 0 0" rpy="0 0 0" />
           <geometry>
-            <mesh filename="package://unity_robot_description/models/robotiq/robotiq_2f_85/visual/robotiq_arg2f_base_link.stl" />
-          </geometry>
-          <material name="">
-            <color rgba="0.1 0.1 0.1 1" />
-          </material>
-        </visual>
-        <collision>
-          <origin xyz="0 0 0" rpy="0 0 0" />
-          <geometry>
-            <mesh filename="package://unity_robot_description/models/robotiq/robotiq_2f_85/collision/robotiq_arg2f_base_link.stl" />
+            <mesh filename="package://ur_remote_control/models/robotiq_2f_85/visual/robotiq_arg2f_base_link.stl" />
+          </geometry>
+          <material name="">
+            <color rgba="0.1 0.1 0.1 1" />
+          </material>
+        </visual>
+        <collision>
+          <origin xyz="0 0 0" rpy="0 0 0" />
+          <geometry>
+            <mesh filename="package://ur_remote_control/models/robotiq_2f_85/collision/robotiq_arg2f_base_link.stl" />
           </geometry>
         </collision>

File: catkin_ws/src/ur_remote_control/urdf/macros/ur5e_macro.xacro (robot description, xacro)
@@ -19,8 +19,8 @@
   <xacro:macro name="ur5e_robot" params="
    prefix
-   joint_limits_parameters_file:='$(find unity_robot_description)/configs/ur5e/joint_limits.yaml'
-   kinematics_parameters_file:='$(find unity_robot_description)/configs/ur5e/default_kinematics.yaml'
-   physical_parameters_file:='$(find unity_robot_description)/configs/ur5e/physical_parameters.yaml'
-   visual_parameters_file:='$(find unity_robot_description)/configs/ur5e/visual_parameters.yaml'
+   joint_limits_parameters_file:='$(find ur_remote_control)/configs/ur5e/joint_limits.yaml'
+   kinematics_parameters_file:='$(find ur_remote_control)/configs/ur5e/default_kinematics.yaml'
+   physical_parameters_file:='$(find ur_remote_control)/configs/ur5e/physical_parameters.yaml'
+   visual_parameters_file:='$(find ur_remote_control)/configs/ur5e/visual_parameters.yaml'
    transmission_hw_interface:=hardware_interface/PositionJointInterface
    safety_limits:=false
@@ -28,5 +28,5 @@
    safety_k_position:=20"
   >
-    <xacro:include filename="$(find unity_robot_description)/xacro/macros/ur_macro.xacro"/>
+    <xacro:include filename="$(find ur_remote_control)/urdf/macros/ur_macro.xacro"/>
     <xacro:ur_robot
       prefix="${prefix}"

File: catkin_ws/src/ur_remote_control/urdf/macros/ur_macro.xacro (robot description, xacro)
@@ -42,6 +42,6 @@
      - Muhammad Asif Rana
   -->
-  <xacro:include filename="$(find unity_robot_description)/xacro/macros/ur_transmissions.xacro" />
-  <xacro:include filename="$(find unity_robot_description)/xacro/macros/ur_common.xacro" />
+  <xacro:include filename="$(find ur_remote_control)/urdf/macros/ur_transmissions.xacro" />
+  <xacro:include filename="$(find ur_remote_control)/urdf/macros/ur_common.xacro" />
   <xacro:macro name="ur_robot" params="
     prefix

File: catkin_ws/src/ur_remote_control/urdf/macros/usb_plug.xacro (robot description, xacro)
@@ -20,5 +20,5 @@
         <geometry>
           <!--box size="0.044850 0.008 0.0185" /-->
-          <mesh filename="package://unity_robot_description/models/intel_realsense/plug.stl" />
+          <mesh filename="package://ur_remote_control/models/l515/plug.stl" />
         </geometry>
         <material name="plastic"/>
@@ -28,5 +28,5 @@
         <geometry>
           <!--box size="0.044850 0.008 0.0185" /-->
-          <mesh filename="package://unity_robot_description/models/intel_realsense/plug_collision.stl" />
+          <mesh filename="package://ur_remote_control/models/l515/plug_collision.stl" />
         </geometry>
       </collision>
