Commit message: added nomenclature description for renaming

File: catkin_ws/src/rvl_robot_description/xacro/robotiq/include/robotiq_2f_common.xacro (robot description, xacro)
@@ -1,3 +1,9 @@
 <?xml version="1.0"?>
 <robot xmlns:xacro="http://www.ros.org/wiki/xacro">
+    <xacro:macro name="load_robotiq_config" params="joint_config_parameters_file physical_parameters_file visual_parameters_file">
+        <!-- Read .yaml files from disk, load content into properties -->
+        <xacro:property name="config_joint_config_parameters" value="${xacro.load_yaml(joint_config_parameters_file)}" />
+        <xacro:property name="config_physical_parameters" value="${xacro.load_yaml(physical_parameters_file)}" />
+        <xacro:property name="config_visual_parameters" value="${xacro.load_yaml(visual_parameters_file)}" />
+    </xacro:macro>
 </robot>

File: catkin_ws/src/rvl_robot_description/xacro/robotiq/include/robotiq_2f_macro.xacro (robot description, xacro)
@@ -1,3 +1,5 @@
 <?xml version="1.0"?>
 <robot xmlns:xacro="http://www.ros.org/wiki/xacro">
+    <xacro:macro name="robotiq_2f_palm" params="prefix">
+    </xacro:macro>
 </robot>
