Commit message: working 2F loading and viewing

File: catkin_ws/src/rvl_robot_description/xacro/robotiq/include/robotiq_2f_transmissions.xacro (robot description, xacro)
@@ -1,3 +1,14 @@
 <?xml version="1.0"?>
-<robot xmlns:xacro="http://www.ros.org/wiki/xacro">
+<robot xmlns:xacro="http://ros.org/wiki/xacro">
+    <xacro:macro name="robotiq_2f_transmission" params="prefix hw_interface">
+        <transmission name="${prefix}finger_joint_trans">
+            <type>transmission_interface/SimpleTransmission</type>
+            <joint name="${prefix}finger_joint">
+                <hardwareInterface>${hw_interface}</hardwareInterface>
+            </joint>
+            <actuator name="${prefix}finger_joint_motor">
+                <mechanicalReduction>1</mechanicalReduction>
+            </actuator>
+        </transmission>
+    </xacro:macro>
 </robot>

File: catkin_ws/src/rvl_robot_description/xacro/robotiq/robotiq_arg2f_140.xacro (robot description, xacro)
@@ -1,11 +1,9 @@
 <?xml version="1.0"?>
 <robot name="robotiq_arg2f_140_model" xmlns:xacro="http://ros.org/wiki/xacro">
-   <!-- import main macro -->
-  <xacro:include filename="$(find robotiq_2f_140_gripper_visualization)/urdf/robotiq_arg2f_140_macro.xacro" />
-  <!-- parameters -->
-  <xacro:arg name="transmission_hw_interface" default="hardware_interface/EffortJointInterface"/>
-  <!-- gripper -->
-  <xacro:robotiq_arg2f_140
-    prefix=""
-    transmission_hw_interface="$(arg transmission_hw_interface)"/>
+    <!-- import main macro -->
+    <xacro:include filename="$(find rvl_robot_description)/xacro/robotiq/include/robotiq_arg2f_140_macro.xacro" />
+    <!-- parameters -->
+    <xacro:arg name="transmission_hw_interface" default="hardware_interface/EffortJointInterface" />
+    <!-- gripper -->
+    <xacro:robotiq_arg2f_140 prefix="" transmission_hw_interface="$(arg transmission_hw_interface)" />
 </robot>

File: catkin_ws/src/rvl_robot_description/xacro/robotiq/robotiq_arg2f_85.xacro (robot description, xacro)
@@ -1,11 +1,9 @@
 <?xml version="1.0"?>
 <robot name="robotiq_arg2f_85_model" xmlns:xacro="http://ros.org/wiki/xacro">
-   <!-- import main macro -->
-  <xacro:include filename="$(find robotiq_2f_85_gripper_visualization)/urdf/robotiq_arg2f_85_macro.xacro" />
-  <!-- parameters -->
-  <xacro:arg name="transmission_hw_interface" default="hardware_interface/EffortJointInterface"/>
-  <!-- gripper -->
-  <xacro:robotiq_arg2f_85
-    prefix=""
-    transmission_hw_interface="$(arg transmission_hw_interface)"/>
+    <!-- import main macro -->
+    <xacro:include filename="$(find rvl_robot_description)/xacro/robotiq/include/robotiq_arg2f_85_macro.xacro" />
+    <!-- parameters -->
+    <xacro:arg name="transmission_hw_interface" default="hardware_interface/EffortJointInterface" />
+    <!-- gripper -->
+    <xacro:robotiq_arg2f_85 prefix="" transmission_hw_interface="$(arg transmission_hw_interface)" />
 </robot>
