Commit message: added Robotiq 2F and 3F models and macros

File: catkin_ws/src/rvl_robot_description/xacro/robotiq/include/robotiq_2f_macro.xacro (robot description, xacro)
@@ -1,5 +1,3 @@
 <?xml version="1.0"?>
 <robot xmlns:xacro="http://www.ros.org/wiki/xacro">
-    <xacro:macro name="robotiq_2f_palm" params="prefix">
-    </xacro:macro>
 </robot>

Commit message: allow robotiq gripper attachment

File: catkin_ws/src/rvl_robot_description/xacro/robotiq/include/robotiq_2f_macro.xacro (robot description, xacro)
@@ -3,5 +3,15 @@
     <xacro:include filename="$(find rvl_robot_description)/xacro/robotiq/include/robotiq_2f_transmissions.xacro" />
     <xacro:include filename="$(find rvl_robot_description)/xacro/robotiq/include/robotiq_2f_common.xacro" />
-    <xacro:macro name="robotiq_2f_gripper" params="prefix stroke transmission_hw_interface:=hardware_interface/EffortJointInterface">
+    <xacro:macro name="robotiq_2f_gripper" params="
+        prefix
+        stroke
+        transmission_hw_interface:=hardware_interface/EffortJointInterface
+        parent_link:=''
+        attachment_x:=0.0
+        attachment_y:=0.0
+        attachment_z:=0.0
+        attachment_roll:=0.0
+        attachment_pitch:=0.0
+        attachment_yaw:=0.0">
         <!-- load stroke-specified configurations -->
         <xacro:load_robotiq_config joint_parameters_file="$(find rvl_robot_description)/config/robotiq/2f_${stroke}/joint_parameters.yaml" physical_parameters_file="$(find rvl_robot_description)/config/robotiq/2f_${stroke}/physical_parameters.yaml" visual_parameters_file="$(find rvl_robot_description)/config/robotiq/2f_${stroke}/visual_parameters.yaml" />
@@ -229,4 +239,20 @@
             <mimic joint="${prefix}${mimic_knuckle_joint_mimic_joint}" multiplier="${mimic_knuckle_joint_mimic_multiplier}" offset="${mimic_knuckle_joint_mimic_offset}" />
         </joint>
+        <!-- ATTACHMENT WHEN REQUIRED -->
+        <xacro:if value="${parent_link != ''}">
+            <joint name="robotiq_2f_to_parent" type="fixed">
+                <parent link="${parent_link}"/>
+                <child link="${prefix}${palm_link_name}"/>
+                <origin xyz="${attachment_x} ${attachment_y} ${attachment_z}" rpy="${attachment_roll} ${attachment_pitch} ${attachment_yaw}"/>
+            </joint>
+        </xacro:if>
+        <xacro:if value="${parent_link == ''}">
+            <link name="base_link"/>
+            <joint name="robotiq_2f_to_parent" type="fixed">
+                <parent link="base_link"/>
+                <child link="${prefix}${palm_link_name}"/>
+                <origin xyz="${attachment_x} ${attachment_y} ${attachment_z}" rpy="${attachment_roll} ${attachment_pitch} ${attachment_yaw}"/>
+            </joint>
+        </xacro:if>
     </xacro:macro>
 </robot>

File: catkin_ws/src/rvl_robot_description/xacro/universal_robots/ur_robot.xacro (robot description, xacro)
@@ -1,23 +1,24 @@
 <?xml version="1.0"?>
 <robot xmlns:xacro="http://wiki.ros.org/xacro" name="ur_robot">
-  <!--
+    <!--
     This is unified Universal Robot macro example instead of individual loading files
     like official ur_description repository.
     Available variants are ur3(e), ur5(e), ur10(e), and ur16e
   -->
-  <xacro:include filename="$(find rvl_robot_description)/xacro/universal_robots/include/ur_macro.xacro"/>
-  <!-- default parameters as before -->
-  <xacro:arg name="transmission_hw_interface" default="hardware_interface/PositionJointInterface"/>
-  <xacro:arg name="safety_limits" default="false"/>
-  <xacro:arg name="safety_pos_margin" default="0.15"/>
-  <xacro:arg name="safety_k_position" default="20"/>
-  <!-- robot model must be specified -->
-  <xacro:arg name="ur_variant" default="ur5e"/>
-  <xacro:ur_robot
-    prefix=""
-    variant="$(arg ur_variant)"
-    transmission_hw_interface="$(arg transmission_hw_interface)"
-    safety_limits="$(arg safety_limits)"
-    safety_pos_margin="$(arg safety_pos_margin)"
-    safety_k_position="$(arg safety_k_position)"/>
+    <xacro:include filename="$(find rvl_robot_description)/xacro/universal_robots/include/ur_macro.xacro" />
+    <!-- default parameters as before -->
+    <xacro:arg name="transmission_hw_interface" default="hardware_interface/PositionJointInterface" />
+    <xacro:arg name="safety_limits" default="false" />
+    <xacro:arg name="safety_pos_margin" default="0.15" />
+    <xacro:arg name="safety_k_position" default="20" />
+    <!-- robot model must be specified -->
+    <xacro:arg name="ur_variant" default="ur5e" />
+    <!-- instantiate the robot -->
+    <xacro:ur_robot
+        prefix=""
+        variant="$(arg ur_variant)"
+        transmission_hw_interface="$(arg transmission_hw_interface)"
+        safety_limits="$(arg safety_limits)"
+        safety_pos_margin="$(arg safety_pos_margin)"
+        safety_k_position="$(arg safety_k_position)" />
 </robot>
