Commit message: combined UR xacro

File: catkin_ws/src/rvl_robot_description/xacro/universal_robots/include/ur_macro.xacro (robot description, xacro)
@@ -1,319 +1,305 @@
 <?xml version="1.0"?>
 <robot xmlns:xacro="http://wiki.ros.org/xacro">
-  <!--
-    Base UR robot series xacro macro.
-    NOTE: this is NOT a URDF. It cannot directly be loaded by consumers
-    expecting a flattened '.urdf' file. See the top-level '.xacro' for that
-    (but note: that .xacro must still be processed by the xacro command).
-    For use in '.launch' files: use one of the 'load_urX.launch' convenience
-    launch files.
-    This file models the base kinematic chain of a UR robot, which then gets
-    parameterised by various configuration files to convert it into a UR3(e),
-    UR5(e), UR10(e) or UR16e.
-    NOTE: the default kinematic parameters (ie: link lengths, frame locations,
-    offets, etc) do not correspond to any particular robot. They are defaults
-    only. There WILL be non-zero offsets between the Forward Kinematics results
-    in TF (ie: robot_state_publisher) and the values reported by the Teach
-    Pendant.
-    For accurate (and robot-specific) transforms, the 'kinematics_parameters_file'
-    parameter MUST point to a .yaml file containing the appropriate values for
-    the targetted robot.
-    If using the UniversalRobots/Universal_Robots_ROS_Driver, follow the steps
-    described in the readme of that repository to extract the kinematic
-    calibration from the controller and generate the required .yaml file.
-    Main author of the migration to yaml configs: Ludovic Delval.
-    Contributors to previous versions (in no particular order):
-     - Felix Messmer
-     - Kelsey Hawkins
-     - Wim Meeussen
-     - Shaun Edwards
-     - Nadia Hammoudeh Garcia
-     - Dave Hershberger
-     - G. vd. Hoorn
-     - Philip Long
-     - Dave Coleman
-     - Miguel Prada
-     - Mathias Luedtke
-     - Marcel Schnirring
-     - Felix von Drigalski
-     - Felix Exner
-     - Jimmy Da Silva
-     - Ajit Krisshna N L
-     - Muhammad Asif Rana
-  -->
-  <xacro:include filename="$(find rvl_robot_description)/xacro/universal_robots/include/ur_transmissions.xacro" />
-  <xacro:include filename="$(find rvl_robot_description)/xacro/universal_robots/include/ur_common.xacro" />
-  <xacro:macro name="ur_robot" params="
-    prefix
-    joint_limits_parameters_file
-    kinematics_parameters_file
-    physical_parameters_file
-    visual_parameters_file
-    transmission_hw_interface:=hardware_interface/PositionJointInterface
-    safety_limits:=false
-    safety_pos_margin:=0.15
-    safety_k_position:=20"
-  >
-    <!-- Load configuration data from the provided .yaml files -->
-    <xacro:read_model_data
-      joint_limits_parameters_file="${joint_limits_parameters_file}"
-      kinematics_parameters_file="${kinematics_parameters_file}"
-      physical_parameters_file="${physical_parameters_file}"
-      visual_parameters_file="${visual_parameters_file}"/>
-    <!-- Add URDF transmission elements (for ros_control) -->
-    <xacro:ur_arm_transmission prefix="${prefix}" hw_interface="${transmission_hw_interface}" />
-    <!-- links: main serial chain -->
-    <link name="${prefix}base_link"/>
-    <link name="${prefix}base_link_inertia">
-      <visual>
-        <origin xyz="0 0 0" rpy="0 0 ${pi}"/>
-        <geometry>
-          <mesh filename="${base_visual_mesh}"/>
-        </geometry>
-        <material name="${base_visual_material_name}">
-          <color rgba="${base_visual_material_color}"/>
-        </material>
-      </visual>
-      <collision>
-        <origin xyz="0 0 0" rpy="0 0 ${pi}"/>
-        <geometry>
-          <mesh filename="${base_collision_mesh}"/>
-        </geometry>
-      </collision>
-      <xacro:cylinder_inertial radius="${base_inertia_radius}" length="${base_inertia_length}" mass="${base_mass}">
-        <origin xyz="0 0 0" rpy="0 0 0" />
-      </xacro:cylinder_inertial>
-    </link>
-    <link name="${prefix}shoulder_link">
-      <visual>
-        <origin xyz="0 0 0" rpy="0 0 ${pi}"/>
-        <geometry>
-          <mesh filename="${shoulder_visual_mesh}"/>
-        </geometry>
-        <material name="${shoulder_visual_material_name}">
-          <color rgba="${shoulder_visual_material_color}"/>
-        </material>
-      </visual>
-      <collision>
-        <origin xyz="0 0 0" rpy="0 0 ${pi}"/>
-        <geometry>
-          <mesh filename="${shoulder_collision_mesh}"/>
-        </geometry>
-      </collision>
-      <xacro:cylinder_inertial radius="${shoulder_inertia_radius}" length="${shoulder_inertia_length}" mass="${shoulder_mass}">
-        <origin xyz="0 0 0" rpy="0 0 0" />
-      </xacro:cylinder_inertial>
-    </link>
-    <link name="${prefix}upper_arm_link">
-      <visual>
-        <origin xyz="0 0 ${shoulder_offset}" rpy="${pi/2} 0 ${-pi/2}"/>
-        <geometry>
-          <mesh filename="${upper_arm_visual_mesh}"/>
-        </geometry>
-        <material name="${upper_arm_visual_material_name}">
-          <color rgba="${upper_arm_visual_material_color}"/>
-        </material>
-      </visual>
-      <collision>
-        <origin xyz="0 0 ${shoulder_offset}" rpy="${pi/2} 0 ${-pi/2}"/>
-        <geometry>
-          <mesh filename="${upper_arm_collision_mesh}"/>
-        </geometry>
-      </collision>
-      <xacro:cylinder_inertial radius="${upperarm_inertia_radius}" length="${upperarm_inertia_length}" mass="${upper_arm_mass}">
-        <origin xyz="${-0.5 * upperarm_inertia_length} 0.0 ${upper_arm_inertia_offset}" rpy="0 ${pi/2} 0" />
-      </xacro:cylinder_inertial>
-    </link>
-    <link name="${prefix}forearm_link">
-      <visual>
-        <origin xyz="0 0 ${elbow_offset}" rpy="${pi/2} 0 ${-pi/2}"/>
-        <geometry>
-          <mesh filename="${forearm_visual_mesh}"/>
-        </geometry>
-        <material name="${forearm_visual_material_name}">
-          <color rgba="${forearm_visual_material_color}"/>
-        </material>
-      </visual>
-      <collision>
-        <origin xyz="0 0 ${elbow_offset}" rpy="${pi/2} 0 ${-pi/2}"/>
-        <geometry>
-          <mesh filename="${forearm_collision_mesh}"/>
-        </geometry>
-      </collision>
-      <xacro:cylinder_inertial radius="${forearm_inertia_radius}" length="${forearm_inertia_length}"  mass="${forearm_mass}">
-        <origin xyz="${-0.5 * forearm_inertia_length} 0.0 ${elbow_offset}" rpy="0 ${pi/2} 0" />
-      </xacro:cylinder_inertial>
-    </link>
-    <link name="${prefix}wrist_1_link">
-      <visual>
-        <!-- TODO: Move this to a parameter -->
-        <origin xyz="0 0 ${wrist_1_visual_offset}" rpy="${pi/2} 0 0"/>
-        <geometry>
-          <mesh filename="${wrist_1_visual_mesh}"/>
-        </geometry>
-        <material name="${wrist_1_visual_material_name}">
-          <color rgba="${wrist_1_visual_material_color}"/>
-        </material>
-      </visual>
-      <collision>
-        <origin xyz="0 0 ${wrist_1_visual_offset}" rpy="${pi/2} 0 0"/>
-        <geometry>
-          <mesh filename="${wrist_1_collision_mesh}"/>
-        </geometry>
-      </collision>
-      <xacro:cylinder_inertial radius="${wrist_1_inertia_radius}" length="${wrist_1_inertia_length}"  mass="${wrist_1_mass}">
-        <origin xyz="0 0 0" rpy="0 0 0" />
-      </xacro:cylinder_inertial>
-    </link>
-    <link name="${prefix}wrist_2_link">
-      <visual>
-        <origin xyz="0 0 ${wrist_2_visual_offset}" rpy="0 0 0"/>
-        <geometry>
-          <mesh filename="${wrist_2_visual_mesh}"/>
-        </geometry>
-        <material name="${wrist_2_visual_material_name}">
-          <color rgba="${wrist_2_visual_material_color}"/>
-        </material>
-      </visual>
-      <collision>
-        <origin xyz="0 0 ${wrist_2_visual_offset}" rpy="0 0 0"/>
-        <geometry>
-          <mesh filename="${wrist_2_collision_mesh}"/>
-        </geometry>
-      </collision>
-      <xacro:cylinder_inertial radius="${wrist_2_inertia_radius}" length="${wrist_2_inertia_length}"  mass="${wrist_2_mass}">
-        <origin xyz="0 0 0" rpy="0 0 0" />
-      </xacro:cylinder_inertial>
-    </link>
-    <link name="${prefix}wrist_3_link">
-      <visual>
-        <origin xyz="0 0 ${wrist_3_visual_offset}" rpy="${pi/2} 0 0"/>
-        <geometry>
-          <mesh filename="${wrist_3_visual_mesh}"/>
-        </geometry>
-        <material name="${wrist_3_visual_material_name}">
-          <color rgba="${wrist_3_visual_material_color}"/>
-        </material>
-      </visual>
-      <collision>
-        <origin xyz="0 0 ${wrist_3_visual_offset}" rpy="${pi/2} 0 0"/>
-        <geometry>
-          <mesh filename="${wrist_3_collision_mesh}"/>
-        </geometry>
-      </collision>
-      <xacro:cylinder_inertial radius="${wrist_3_inertia_radius}" length="${wrist_3_inertia_length}"  mass="${wrist_3_mass}">
-        <origin xyz="0.0 0.0 ${-0.5 * wrist_3_inertia_length}" rpy="0 0 0" />
-      </xacro:cylinder_inertial>
-    </link>
-    <!-- joints: main serial chain -->
-    <joint name="${prefix}base_link-base_link_inertia" type="fixed">
-      <parent link="${prefix}base_link" />
-      <child link="${prefix}base_link_inertia" />
-      <!-- 'base_link' is REP-103 aligned (so X+ forward), while the internal
+    <!--
+        Base UR robot series xacro macro.
+        NOTE: this is NOT a URDF. It cannot directly be loaded by consumers
+        expecting a flattened '.urdf' file. See the top-level '.xacro' for that
+        (but note: that .xacro must still be processed by the xacro command).
+        For use in '.launch' files: use one of the 'load_urX.launch' convenience
+        launch files.
+        This file models the base kinematic chain of a UR robot, which then gets
+        parameterised by various configuration files to convert it into a UR3(e),
+        UR5(e), UR10(e) or UR16e.
+        NOTE: the default kinematic parameters (ie: link lengths, frame locations,
+        offets, etc) do not correspond to any particular robot. They are defaults
+        only. There WILL be non-zero offsets between the Forward Kinematics results
+        in TF (ie: robot_state_publisher) and the values reported by the Teach
+        Pendant.
+        For accurate (and robot-specific) transforms, the 'kinematics_parameters_file'
+        parameter MUST point to a .yaml file containing the appropriate values for
+        the targetted robot.
+        If using the UniversalRobots/Universal_Robots_ROS_Driver, follow the steps
+        described in the readme of that repository to extract the kinematic
+        calibration from the controller and generate the required .yaml file.
+        Main author of the migration to yaml configs: Ludovic Delval.
+        Contributors to previous versions (in no particular order):
+        - Felix Messmer
+        - Kelsey Hawkins
+        - Wim Meeussen
+        - Shaun Edwards
+        - Nadia Hammoudeh Garcia
+        - Dave Hershberger
+        - G. vd. Hoorn
+        - Philip Long
+        - Dave Coleman
+        - Miguel Prada
+        - Mathias Luedtke
+        - Marcel Schnirring
+        - Felix von Drigalski
+        - Felix Exner
+        - Jimmy Da Silva
+        - Ajit Krisshna N L
+        - Muhammad Asif Rana
+    -->
+    <xacro:include filename="$(find rvl_robot_description)/xacro/universal_robots/include/ur_transmissions.xacro" />
+    <xacro:include filename="$(find rvl_robot_description)/xacro/universal_robots/include/ur_common.xacro" />
+    <xacro:macro name="ur_robot" params="
+        prefix
+        variant
+        transmission_hw_interface:=hardware_interface/PositionJointInterface
+        safety_limits:=false
+        safety_pos_margin:=0.15
+        safety_k_position:=20">
+        <!-- Load configuration data from the provided .yaml files -->
+        <xacro:read_model_data joint_limits_parameters_file="$(find rvl_robot_description)/config/universal_robots/${variant}/joint_limits.yaml" kinematics_parameters_file="$(find rvl_robot_description)/config/universal_robots/${variant}/default_kinematics.yaml" physical_parameters_file="$(find rvl_robot_description)/config/universal_robots/${variant}/physical_parameters.yaml" visual_parameters_file="$(find rvl_robot_description)/config/universal_robots/${variant}/visual_parameters.yaml" />
+        <!-- Add URDF transmission elements (for ros_control) -->
+        <xacro:ur_arm_transmission prefix="${prefix}" hw_interface="${transmission_hw_interface}" />
+        <!-- links: main serial chain -->
+        <link name="${prefix}base_link" />
+        <link name="${prefix}base_link_inertia">
+            <visual>
+                <origin xyz="0 0 0" rpy="0 0 ${pi}" />
+                <geometry>
+                    <mesh filename="${base_visual_mesh}" />
+                </geometry>
+                <material name="${base_visual_material_name}">
+                    <color rgba="${base_visual_material_color}" />
+                </material>
+            </visual>
+            <collision>
+                <origin xyz="0 0 0" rpy="0 0 ${pi}" />
+                <geometry>
+                    <mesh filename="${base_collision_mesh}" />
+                </geometry>
+            </collision>
+            <xacro:cylinder_inertial radius="${base_inertia_radius}" length="${base_inertia_length}" mass="${base_mass}">
+                <origin xyz="0 0 0" rpy="0 0 0" />
+            </xacro:cylinder_inertial>
+        </link>
+        <link name="${prefix}shoulder_link">
+            <visual>
+                <origin xyz="0 0 0" rpy="0 0 ${pi}" />
+                <geometry>
+                    <mesh filename="${shoulder_visual_mesh}" />
+                </geometry>
+                <material name="${shoulder_visual_material_name}">
+                    <color rgba="${shoulder_visual_material_color}" />
+                </material>
+            </visual>
+            <collision>
+                <origin xyz="0 0 0" rpy="0 0 ${pi}" />
+                <geometry>
+                    <mesh filename="${shoulder_collision_mesh}" />
+                </geometry>
+            </collision>
+            <xacro:cylinder_inertial radius="${shoulder_inertia_radius}" length="${shoulder_inertia_length}" mass="${shoulder_mass}">
+                <origin xyz="0 0 0" rpy="0 0 0" />
+            </xacro:cylinder_inertial>
+        </link>
+        <link name="${prefix}upper_arm_link">
+            <visual>
+                <origin xyz="0 0 ${shoulder_offset}" rpy="${pi/2} 0 ${-pi/2}" />
+                <geometry>
+                    <mesh filename="${upper_arm_visual_mesh}" />
+                </geometry>
+                <material name="${upper_arm_visual_material_name}">
+                    <color rgba="${upper_arm_visual_material_color}" />
+                </material>
+            </visual>
+            <collision>
+                <origin xyz="0 0 ${shoulder_offset}" rpy="${pi/2} 0 ${-pi/2}" />
+                <geometry>
+                    <mesh filename="${upper_arm_collision_mesh}" />
+                </geometry>
+            </collision>
+            <xacro:cylinder_inertial radius="${upperarm_inertia_radius}" length="${upperarm_inertia_length}" mass="${upper_arm_mass}">
+                <origin xyz="${-0.5 * upperarm_inertia_length} 0.0 ${upper_arm_inertia_offset}" rpy="0 ${pi/2} 0" />
+            </xacro:cylinder_inertial>
+        </link>
+        <link name="${prefix}forearm_link">
+            <visual>
+                <origin xyz="0 0 ${elbow_offset}" rpy="${pi/2} 0 ${-pi/2}" />
+                <geometry>
+                    <mesh filename="${forearm_visual_mesh}" />
+                </geometry>
+                <material name="${forearm_visual_material_name}">
+                    <color rgba="${forearm_visual_material_color}" />
+                </material>
+            </visual>
+            <collision>
+                <origin xyz="0 0 ${elbow_offset}" rpy="${pi/2} 0 ${-pi/2}" />
+                <geometry>
+                    <mesh filename="${forearm_collision_mesh}" />
+                </geometry>
+            </collision>
+            <xacro:cylinder_inertial radius="${forearm_inertia_radius}" length="${forearm_inertia_length}" mass="${forearm_mass}">
+                <origin xyz="${-0.5 * forearm_inertia_length} 0.0 ${elbow_offset}" rpy="0 ${pi/2} 0" />
+            </xacro:cylinder_inertial>
+        </link>
+        <link name="${prefix}wrist_1_link">
+            <visual>
+                <!-- TODO: Move this to a parameter -->
+                <origin xyz="0 0 ${wrist_1_visual_offset}" rpy="${pi/2} 0 0" />
+                <geometry>
+                    <mesh filename="${wrist_1_visual_mesh}" />
+                </geometry>
+                <material name="${wrist_1_visual_material_name}">
+                    <color rgba="${wrist_1_visual_material_color}" />
+                </material>
+            </visual>
+            <collision>
+                <origin xyz="0 0 ${wrist_1_visual_offset}" rpy="${pi/2} 0 0" />
+                <geometry>
+                    <mesh filename="${wrist_1_collision_mesh}" />
+                </geometry>
+            </collision>
+            <xacro:cylinder_inertial radius="${wrist_1_inertia_radius}" length="${wrist_1_inertia_length}" mass="${wrist_1_mass}">
+                <origin xyz="0 0 0" rpy="0 0 0" />
+            </xacro:cylinder_inertial>
+        </link>
+        <link name="${prefix}wrist_2_link">
+            <visual>
+                <origin xyz="0 0 ${wrist_2_visual_offset}" rpy="0 0 0" />
+                <geometry>
+                    <mesh filename="${wrist_2_visual_mesh}" />
+                </geometry>
+                <material name="${wrist_2_visual_material_name}">
+                    <color rgba="${wrist_2_visual_material_color}" />
+                </material>
+            </visual>
+            <collision>
+                <origin xyz="0 0 ${wrist_2_visual_offset}" rpy="0 0 0" />
+                <geometry>
+                    <mesh filename="${wrist_2_collision_mesh}" />
+                </geometry>
+            </collision>
+            <xacro:cylinder_inertial radius="${wrist_2_inertia_radius}" length="${wrist_2_inertia_length}" mass="${wrist_2_mass}">
+                <origin xyz="0 0 0" rpy="0 0 0" />
+            </xacro:cylinder_inertial>
+        </link>
+        <link name="${prefix}wrist_3_link">
+            <visual>
+                <origin xyz="0 0 ${wrist_3_visual_offset}" rpy="${pi/2} 0 0" />
+                <geometry>
+                    <mesh filename="${wrist_3_visual_mesh}" />
+                </geometry>
+                <material name="${wrist_3_visual_material_name}">
+                    <color rgba="${wrist_3_visual_material_color}" />
+                </material>
+            </visual>
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