Commit message: working modular RVL UR arm definition

File: catkin_ws/src/rvl_robot_description/xacro/custom/mounting_plate.xacro (robot description, xacro)
@@ -26,4 +26,4 @@
     </xacro:macro>
     <!-- testing -->
-    <xacro:L515_mounting_plate prefix="" />
+    <!-- <xacro:L515_mounting_plate prefix="" /> -->
 </robot>

File: catkin_ws/src/rvl_robot_description/xacro/robotiq/include/robotiq_2f_macro.xacro (robot description, xacro)
@@ -15,5 +15,8 @@
         attachment_yaw:=0.0">
         <!-- load stroke-specified configurations -->
-        <xacro:load_robotiq_config joint_parameters_file="$(find rvl_robot_description)/config/robotiq/2f_${stroke}/joint_parameters.yaml" physical_parameters_file="$(find rvl_robot_description)/config/robotiq/2f_${stroke}/physical_parameters.yaml" visual_parameters_file="$(find rvl_robot_description)/config/robotiq/2f_${stroke}/visual_parameters.yaml" />
+        <xacro:load_robotiq_config
+            joint_parameters_file="$(find rvl_robot_description)/config/robotiq/2f_${stroke}/joint_parameters.yaml"
+            physical_parameters_file="$(find rvl_robot_description)/config/robotiq/2f_${stroke}/physical_parameters.yaml"
+            visual_parameters_file="$(find rvl_robot_description)/config/robotiq/2f_${stroke}/visual_parameters.yaml" />
         <!-- attached hardware interface for ros_control -->
         <xacro:robotiq_2f_transmission prefix="${prefix}" hw_interface="${transmission_hw_interface}" driven_joint="${prefix}${knuckle_joint_name}" />
@@ -241,5 +244,5 @@
         <!-- ATTACHMENT WHEN REQUIRED -->
         <xacro:if value="${parent_link != ''}">
-            <joint name="robotiq_2f_to_parent" type="fixed">
+            <joint name="${parent_link}-robotiq_2f_base" type="fixed">
                 <parent link="${parent_link}"/>
                 <child link="${prefix}${palm_link_name}"/>
