Commit message: working unified Robotiq 2F description

File: catkin_ws/src/rvl_gazebo/xacro/ur.xacro (robot description, xacro)
@@ -35,9 +35,9 @@
         safety_k_position="$(arg safety_k_position)" />
     <!--
-        Attach the Gazebo model to Gazebo's world frame.
-        Note: if you're looking to integrate a UR into a larger scene and need
-        to add EEFs or other parts, DO NOT change this file or the 'world' link
-        here. Create a NEW xacro instead and decide whether you need to add
-        a 'world' link there.
+    Attach the Gazebo model to Gazebo's world frame.
+    Note: if you're looking to integrate a UR into a larger scene and need
+    to add EEFs or other parts, DO NOT change this file or the 'world' link
+    here. Create a NEW xacro instead and decide whether you need to add
+    a 'world' link there.
     -->
     <link name="world" />

File: catkin_ws/src/rvl_robot_description/xacro/robotiq/include/robotiq_2f_macro.xacro (robot description, xacro)
@@ -164,5 +164,10 @@
         <xacro:macro name="proximal_phalanx_joint" params="prefix fingerprefix reflect">
             <joint name="${prefix}${fingerprefix}${proximal_phalanx_joint_name}" type="${proximal_phalanx_joint_type}">
-                <origin xyz="0 ${reflect * -0.0127} 0.06142" rpy="0 0 ${(1 + reflect) * pi / 2}" />
+                <xacro:if value="${stroke == 85}">
+                    <origin xyz="0 ${reflect * -0.0127} 0.06142" rpy="0 0 ${(1 + reflect) * pi / 2}" />
+                </xacro:if>
+                <xacro:if value="${stroke == 140}">
+                    <origin xyz="0 ${reflect * -0.0127} 0.06142" rpy="${pi / 2 + .725} 0 ${(reflect - 1) * pi / 2}" />
+                </xacro:if>
                 <parent link="${prefix}${proximal_phalanx_joint_parent_link}" />
                 <child link="${prefix}${fingerprefix}${proximal_phalanx_joint_child_link}" />

Commit message: fixed twitchy arm due to naming error

File: catkin_ws/src/rvl_gazebo/xacro/ur.xacro (robot description, xacro)
@@ -7,9 +7,4 @@
     -->
     <xacro:include filename="$(find rvl_gazebo)/xacro/ur_macro.xacro" />
-    <!--Declare arguments -->
-    <xacro:arg name="joint_limit_params" default="" />
-    <xacro:arg name="physical_params" default="" />
-    <xacro:arg name="kinematics_params" default="" />
-    <xacro:arg name="visual_params" default="" />
     <!--
         legal values:
@@ -21,4 +16,5 @@
     -->
     <xacro:arg name="transmission_hw_interface" default="hardware_interface/PositionJointInterface" />
+    <xacro:arg name="variant" default="ur5e" />
     <xacro:arg name="safety_limits" default="false" />
     <xacro:arg name="safety_pos_margin" default="0.15" />
@@ -26,8 +22,5 @@
     <!-- Instantiate the Gazebo robot and pass it all the required arguments. -->
     <xacro:ur_robot_gazebo prefix=""
-        joint_limits_parameters_file="$(arg joint_limit_params)"
-        kinematics_parameters_file="$(arg kinematics_params)"
-        physical_parameters_file="$(arg physical_params)"
-        visual_parameters_file="$(arg visual_params)"
+        variant="$(arg variant)"
         transmission_hw_interface="$(arg transmission_hw_interface)"
         safety_limits="$(arg safety_limits)"

File: catkin_ws/src/rvl_gazebo/xacro/ur_macro.xacro (robot description, xacro)
@@ -4,10 +4,9 @@
     <xacro:macro name="ur_robot_gazebo" params="
         prefix
-        joint_limits_parameters_file
-        kinematics_parameters_file
-        physical_parameters_file
-        visual_parameters_file
+        variant
         transmission_hw_interface:=hardware_interface/PositionJointInterface
-        safety_limits:=false safety_pos_margin:=0.15 safety_k_position:=20">
+        safety_limits:=false
+        safety_pos_margin:=0.15
+        safety_k_position:=20">
         <!--
             Import the xacro macro for the REAL robot (which we'll augment with Gazebo
@@ -18,5 +17,11 @@
         <xacro:include filename="$(find rvl_robot_description)/xacro/universal_robots/include/ur_macro.xacro" />
         <!-- Instantiate model for the REAL robot. -->
-        <xacro:ur_robot prefix="${prefix}" joint_limits_parameters_file="${joint_limits_parameters_file}" kinematics_parameters_file="${kinematics_parameters_file}" physical_parameters_file="${physical_parameters_file}" visual_parameters_file="${visual_parameters_file}" transmission_hw_interface="${transmission_hw_interface}" safety_limits="${safety_limits}" safety_pos_margin="${safety_pos_margin}" safety_k_position="${safety_k_position}" />
+        <xacro:ur_robot
+            prefix="${prefix}"
+            variant="${variant}"
+            transmission_hw_interface="${transmission_hw_interface}"
+            safety_limits="${safety_limits}"
+            safety_pos_margin="${safety_pos_margin}"
+            safety_k_position="${safety_k_position}" />
         <!-- Configure self collision properties per link -->
         <gazebo reference="${prefix}shoulder_link">

File: catkin_ws/src/rvl_robot_description/xacro/robotiq/include/robotiq_2f_common.xacro (robot description, xacro)
@@ -149,6 +149,6 @@
         <!-- INDIVIDUAL JOINT NAMES -->
         <xacro:property name="knuckle_joint_name" value="${sec_joint_names['base_to_knuckle']}" scope="parent" />
-        <xacro:property name="bar_joint_name" value="${sec_joint_names['base_to_proximal']}" scope="parent" />
-        <xacro:property name="proximal_phalanx_joint_name" value="${sec_joint_names['knuckle_to_bar']}" scope="parent" />
+        <xacro:property name="bar_joint_name" value="${sec_joint_names['knuckle_to_bar']}" scope="parent" />
+        <xacro:property name="proximal_phalanx_joint_name" value="${sec_joint_names['base_to_proximal']}" scope="parent" />
         <xacro:property name="distal_phalanx_joint_name" value="${sec_joint_names['bar_to_distal']}" scope="parent" />
         <xacro:property name="finger_tip_joint_name" value="${sec_joint_names['distal_to_tip']}" scope="parent" />

File: catkin_ws/src/rvl_robot_description/xacro/robotiq/include/robotiq_2f_macro.xacro (robot description, xacro)
@@ -222,20 +222,20 @@
         </link>
         <!-- LEFT FINGER -->
-        <xacro:finger_links prefix="${prefix}" fingerprefix="left" />
-        <xacro:finger_joints prefix="${prefix}" fingerprefix="left" reflect="1.0" />
+        <xacro:finger_links prefix="${prefix}" fingerprefix="left_" />
+        <xacro:finger_joints prefix="${prefix}" fingerprefix="left_" reflect="1.0" />
         <joint name="${prefix}${knuckle_joint_name}" type="${knuckle_joint_type}">
             <origin xyz="${knuckle_joint_origin_xyz}" rpy="${knuckle_joint_origin_rpy}" />
             <parent link="${prefix}${knuckle_joint_parent_link}" />
-            <child link="${prefix}left${knuckle_joint_child_link}" />
+            <child link="${prefix}left_${knuckle_joint_child_link}" />
             <axis xyz="${knuckle_joint_axis}" />
             <limit lower="${knuckle_joint_lower_limit}" upper="${knuckle_joint_upper_limit}" velocity="${knuckle_joint_velocity}" effort="${knuckle_joint_effort}" />
         </joint>
         <!-- RIGHT FINGER -->
-        <xacro:finger_links prefix="${prefix}" fingerprefix="right" />
-        <xacro:finger_joints prefix="${prefix}" fingerprefix="right" reflect="-1.0" />
-        <joint name="${prefix}right${knuckle_joint_name}" type="${mimic_knuckle_joint_type}">
+        <xacro:finger_links prefix="${prefix}" fingerprefix="right_" />
+        <xacro:finger_joints prefix="${prefix}" fingerprefix="right_" reflect="-1.0" />
+        <joint name="${prefix}right_${knuckle_joint_name}" type="${mimic_knuckle_joint_type}">
             <origin xyz="${mimic_knuckle_joint_origin_xyz}" rpy="${mimic_knuckle_joint_origin_rpy}" />
             <parent link="${prefix}${mimic_knuckle_joint_parent_link}" />
-            <child link="${prefix}right${mimic_knuckle_joint_child_link}" />
+            <child link="${prefix}right_${mimic_knuckle_joint_child_link}" />
             <axis xyz="${mimic_knuckle_joint_axis}" />
             <limit lower="${mimic_knuckle_joint_lower_limit}" upper="${mimic_knuckle_joint_upper_limit}" velocity="${mimic_knuckle_joint_velocity}" effort="${mimic_knuckle_joint_effort}" />
