Commit message: working MoveIt in Gazebo

File: catkin_ws/src/rvl_gazebo/xacro/rvl_gazebo.xacro (robot description, xacro)
@@ -32,5 +32,5 @@
     <joint name="world_joint" type="fixed">
         <parent link="world" />
-        <child link="base_link" />
+        <child link="$(arg prefix)base_link" />
         <origin xyz="0 0 0" rpy="0 0 0" />
     </joint>

File: catkin_ws/src/rvl_gazebo/xacro/rvl_gazebo_macro.xacro (robot description, xacro)
@@ -19,5 +19,13 @@
         <xacro:arg name="safety_pos_margin" default="0.15" />
         <xacro:arg name="safety_k_position" default="20" />
-        <xacro:rvl_arm prefix="${prefix}" ur_variant="${ur_variant}" ur_transmission_hw_interface="${ur_transmission_hw_interface}" robotiq_variant="${robotiq_variant}" robotiq_transmission_hw_interface="${robotiq_transmission_hw_interface}" safety_limits="${safety_limits}" safety_pos_margin="${safety_pos_margin}" safety_k_position="${safety_k_position}" />
+        <xacro:rvl_arm
+            prefix="${prefix}"
+            ur_variant="${ur_variant}"
+            ur_transmission_hw_interface="${ur_transmission_hw_interface}"
+            robotiq_variant="${robotiq_variant}"
+            robotiq_transmission_hw_interface="${robotiq_transmission_hw_interface}"
+            safety_limits="${safety_limits}"
+            safety_pos_margin="${safety_pos_margin}"
+            safety_k_position="${safety_k_position}" />
         <!-- Configure self collision properties per link -->
         <gazebo reference="${prefix}shoulder_link">

File: catkin_ws/src/rvl_robot_description/xacro/custom/rvl_ur_robotiq_macro.xacro (robot description, xacro)
@@ -39,5 +39,5 @@
                 stroke="${robotiq_variant[3:]}"
                 transmission_hw_interface="${robotiq_transmission_hw_interface}"
-                parent_link="${prefix}L515_mounting_plate"
+                parent_link="${prefix}tool0"
                 attachment_z="${coupling_offset}"
                 attachment_yaw="${tool_rotation}" />

Commit message: simplified Gazebo package

File: catkin_ws/src/rvl_gazebo/xacro/rvl_gazebo.xacro (robot description, xacro)
@@ -1,27 +1,97 @@
 <?xml version="1.0"?>
-<robot xmlns:xacro="http://www.ros.org/wiki/xacro" name="rvl_arm_gazebo">
-    <!-- Include main macro -->
-    <xacro:include filename="$(find rvl_gazebo)/xacro/rvl_gazebo_macro.xacro" />
-    <!-- Default configs, with UR and Robotiq model preset -->
-    <xacro:arg name="prefix" default="" />
-    <xacro:arg name="ur_variant" default="ur5e" />
-    <xacro:arg name="ur_transmission_hw_interface" default="hardware_interface/PositionJointInterface" />
-    <xacro:arg name="robotiq_variant" default="2f_85" />
-    <xacro:arg name="robotiq_transmission_hw_interface" default="hardware_interface/EffortJointInterface" />
-    <xacro:arg name="realsense_variant" default="l515" />
-    <xacro:arg name="safety_limits" default="false" />
-    <xacro:arg name="safety_pos_margin" default="0.15" />
-    <xacro:arg name="safety_k_position" default="20" />
-    <!-- Instantiate the Gazebo robot and pass it all the required arguments. -->
-    <xacro:rvl_arm_gazebo
-        prefix="$(arg prefix)"
-        ur_variant="$(arg ur_variant)"
-        ur_transmission_hw_interface="$(arg ur_transmission_hw_interface)"
-        robotiq_variant="$(arg robotiq_variant)"
-        robotiq_transmission_hw_interface="$(arg robotiq_transmission_hw_interface)"
-        realsense_variant="$(arg realsense_variant)"
-        safety_limits="$(arg safety_limits)"
-        safety_pos_margin="$(arg safety_pos_margin)"
-        safety_k_position="$(arg safety_k_position)" />
+<robot xmlns:xacro="http://www.ros.org/wiki/xacro" name="rvl_ur_gazebo">
+    <xacro:include filename="$(find rvl_robot_description)/xacro/custom/rvl_ur.xacro" />
+    <!-- Configure self collision properties per link -->
+    <gazebo reference="shoulder_link">
+        <selfCollide>true</selfCollide>
+    </gazebo>
+    <gazebo reference="upper_arm_link">
+        <selfCollide>true</selfCollide>
+    </gazebo>
+    <gazebo reference="forearm_link">
+        <selfCollide>true</selfCollide>
+    </gazebo>
+    <gazebo reference="wrist_1_link">
+        <selfCollide>true</selfCollide>
+    </gazebo>
+    <gazebo reference="wrist_3_link">
+        <selfCollide>true</selfCollide>
+    </gazebo>
+    <gazebo reference="wrist_2_link">
+        <selfCollide>true</selfCollide>
+    </gazebo>
+    <gazebo reference="ee_link">
+        <selfCollide>true</selfCollide>
+    </gazebo>
+    <!-- Load joint names from configuration YAML -->
+    <xacro:property name="joint_parameters_file" value="$(find rvl_robot_description)/config/robotiq/2f_85/joint_parameters.yaml" />
+    <xacro:property name="config_joint_parameters" value="${xacro.load_yaml(joint_parameters_file)}" />
+    <xacro:property name="sec_joint_names" value="${config_joint_parameters['joint_names']}" />
+    <xacro:property name="knuckle_joint_name" value="${sec_joint_names['base_to_knuckle']}" />
+    <xacro:property name="bar_joint_name" value="${sec_joint_names['knuckle_to_bar']}" />
+    <xacro:property name="proximal_phalanx_joint_name" value="${sec_joint_names['base_to_proximal']}" />
+    <xacro:property name="distal_phalanx_joint_name" value="${sec_joint_names['bar_to_distal']}" />
+    <xacro:property name="finger_tip_joint_name" value="${sec_joint_names['distal_to_tip']}" />
+    <gazebo>
+        <plugin filename="libroboticsgroup_upatras_gazebo_mimic_joint_plugin.so" name="mimic_robotiq_1">
+            <joint>${knuckle_joint_name}</joint>
+            <mimicJoint>left_${proximal_phalanx_joint_name}</mimicJoint>
+            <multiplier>1.0</multiplier>
+        </plugin>
+        <plugin filename="libroboticsgroup_upatras_gazebo_mimic_joint_plugin.so" name="mimic_robotiq_2">
+            <joint>${knuckle_joint_name}</joint>
+            <mimicJoint>left_${distal_phalanx_joint_name}</mimicJoint>
+            <multiplier>-1.0</multiplier>
+        </plugin>
+        <plugin filename="libroboticsgroup_upatras_gazebo_mimic_joint_plugin.so" name="mimic_robotiq_3">
+            <joint>${knuckle_joint_name}</joint>
+            <mimicJoint>right_${proximal_phalanx_joint_name}</mimicJoint>
+            <multiplier>1.0</multiplier>
+        </plugin>
+        <plugin filename="libroboticsgroup_upatras_gazebo_mimic_joint_plugin.so" name="mimic_robotiq_4">
+            <joint>${knuckle_joint_name}</joint>
+            <mimicJoint>right_${distal_phalanx_joint_name}</mimicJoint>
+            <multiplier>-1.0</multiplier>
+        </plugin>
+        <plugin filename="libroboticsgroup_upatras_gazebo_mimic_joint_plugin.so" name="mimic_robotiq_5">
+            <joint>${knuckle_joint_name}</joint>
+            <mimicJoint>right_${knuckle_joint_name}</mimicJoint>
+            <multiplier>1.0</multiplier>
+        </plugin>
+    </gazebo>
+    <xacro:property name="sec_link_names" value="${config_joint_parameters['link_names']}" />
+    <xacro:property name="palm_link_name" value="${sec_link_names['palm']}" />
+    <xacro:property name="knuckle_link_name" value="${sec_link_names['knuckle']}" />
+    <xacro:property name="bar_link_name" value="${sec_link_names['bar']}" />
+    <xacro:property name="proximal_phalanx_link_name" value="${sec_link_names['proximal_phalanx']}" />
+    <xacro:property name="distal_phalanx_link_name" value="${sec_link_names['distal_phalanx']}" />
+    <xacro:property name="finger_tip_link_name" value="${sec_link_names['finger_tip']}" />
+    <gazebo reference="${palm_link_name}">
+        <material>Gazebo/Black</material>
+    </gazebo>
+    <gazebo reference="left_${knuckle_link_name}">
+        <material>Gazebo/Grey</material>
+    </gazebo>
+    <gazebo reference="left_${bar_link_name}">
+        <material>Gazebo/Black</material>
+    </gazebo>
+    <gazebo reference="left_${proximal_phalanx_link_name}">
+        <material>Gazebo/Grey</material>
+    </gazebo>
+    <gazebo reference="left_${distal_phalanx_link_name}">
+        <material>Gazebo/Black</material>
+    </gazebo>
+    <gazebo reference="right_${knuckle_link_name}">
+        <material>Gazebo/Grey</material>
+    </gazebo>
+    <gazebo reference="right_${bar_link_name}">
+        <material>Gazebo/Black</material>
+    </gazebo>
+    <gazebo reference="right_${proximal_phalanx_link_name}">
+        <material>Gazebo/Grey</material>
+    </gazebo>
+    <gazebo reference="right_${distal_phalanx_link_name}">
+        <material>Gazebo/Black</material>
+    </gazebo>
     <!--
         Attach the Gazebo model to Gazebo's world frame.
@@ -34,6 +104,16 @@
     <joint name="world_joint" type="fixed">
         <parent link="world" />
-        <child link="$(arg prefix)base_link" />
+        <child link="base_link" />
         <origin xyz="0 0 0" rpy="0 0 0" />
     </joint>
+    <!--
+        Inject Gazebo ROS Control plugin, which allows us to use ros_control
+        controllers to control the virtual robot hw.
+    -->
+    <gazebo>
+        <plugin name="ros_control" filename="libgazebo_ros_control.so">
+            <!--robotNamespace>/</robotNamespace-->
+            <!--robotSimType>gazebo_ros_control/DefaultRobotHWSim</robotSimType-->
+        </plugin>
+    </gazebo>
 </robot>

File: catkin_ws/src/rvl_robot_description/xacro/realsense/d455.xacro (robot description, xacro)
@@ -11,5 +11,5 @@
   <xacro:include filename="$(find rvl_robot_description)/xacro/realsense/usb_plug.xacro" />
   <xacro:macro name="sensor_d455" params="parent *origin name:=camera use_nominal_extrinsics:=false">
-    <xacro:arg name="add_plug" default="false" />
+    <xacro:arg name="add_plug" default="true" />
     <xacro:property name="M_PI" value="3.1415926535897931" />
     <!-- The following values are approximate, and the camera node

File: catkin_ws/src/rvl_robot_description/xacro/robotiq/include/robotiq_2f_macro.xacro (robot description, xacro)
@@ -244,5 +244,5 @@
         <!-- ATTACHMENT WHEN REQUIRED -->
         <xacro:if value="${parent_link != ''}">
-            <joint name="${parent_link}-robotiq_2f_base" type="fixed">
+            <joint name="${parent_link}-${palm_link_name}" type="fixed">
                 <parent link="${parent_link}"/>
                 <child link="${prefix}${palm_link_name}"/>

File: catkin_ws/src/rvl_robot_description/xacro/robotiq/robotiq_2f_140.xacro (robot description, xacro)
@@ -1,7 +1,27 @@
 <?xml version="1.0"?>
-<robot xmlns:xacro="http://www.ros.org/wiki/xacro" name="robotiq_2f_85">
+<robot xmlns:xacro="http://www.ros.org/wiki/xacro" name="robotiq_2f_140">
+    <xacro:arg name="prefix" default="" />
+    <xacro:arg name="stroke" default="140" />
+    <xacro:arg name="transmission_hw_interface" default="hardware_interface/EffortJointInterface" />
+    <xacro:arg name="parent_link" default="" />
+    <xacro:arg name="attachment_x" default="0.0" />
+    <xacro:arg name="attachment_y" default="0.0" />
+    <xacro:arg name="attachment_z" default="0.0" />
+    <xacro:arg name="attachment_roll" default="0.0" />
+    <xacro:arg name="attachment_pitch" default="0.0" />
+    <xacro:arg name="attachment_yaw" default="0.0" />
     <!-- import main macro -->
     <xacro:include filename="$(find rvl_robot_description)/xacro/robotiq/include/robotiq_2f_macro.xacro" />
     <!-- gripper -->
-    <xacro:robotiq_2f_gripper prefix="" stroke="140" />
+    <xacro:robotiq_2f_gripper
+        prefix="$(arg prefix)"
+        stroke="$(arg stroke)"
+        transmission_hw_interface="$(arg transmission_hw_interface)"
+        parent_link="$(arg parent_link)"
+        attachment_x="$(arg attachment_x)"
+        attachment_y="$(arg attachment_y)"
+        attachment_z="$(arg attachment_z)"
+        attachment_roll="$(arg attachment_roll)"
+        attachment_pitch="$(arg attachment_pitch)"
+        attachment_yaw="$(arg attachment_yaw)" />
 </robot>

File: catkin_ws/src/rvl_robot_description/xacro/robotiq/robotiq_2f_85.xacro (robot description, xacro)
@@ -1,7 +1,27 @@
 <?xml version="1.0"?>
 <robot xmlns:xacro="http://www.ros.org/wiki/xacro" name="robotiq_2f_85">
+    <xacro:arg name="prefix" default="" />
+    <xacro:arg name="stroke" default="85" />
+    <xacro:arg name="transmission_hw_interface" default="hardware_interface/EffortJointInterface" />
+    <xacro:arg name="parent_link" default="" />
+    <xacro:arg name="attachment_x" default="0.0" />
+    <xacro:arg name="attachment_y" default="0.0" />
+    <xacro:arg name="attachment_z" default="0.0" />
+    <xacro:arg name="attachment_roll" default="0.0" />
+    <xacro:arg name="attachment_pitch" default="0.0" />
+    <xacro:arg name="attachment_yaw" default="0.0" />
     <!-- import main macro -->
     <xacro:include filename="$(find rvl_robot_description)/xacro/robotiq/include/robotiq_2f_macro.xacro" />
     <!-- gripper -->
-    <xacro:robotiq_2f_gripper prefix="" stroke="85" />
+    <xacro:robotiq_2f_gripper
+        prefix="$(arg prefix)"
+        stroke="$(arg stroke)"
+        transmission_hw_interface="$(arg transmission_hw_interface)"
+        parent_link="$(arg parent_link)"
+        attachment_x="$(arg attachment_x)"
+        attachment_y="$(arg attachment_y)"
+        attachment_z="$(arg attachment_z)"
+        attachment_roll="$(arg attachment_roll)"
+        attachment_pitch="$(arg attachment_pitch)"
+        attachment_yaw="$(arg attachment_yaw)" />
 </robot>

File: catkin_ws/src/rvl_robot_description/xacro/universal_robots/include/ur_macro.xacro (robot description, xacro)
@@ -202,9 +202,10 @@
             <parent link="${prefix}base_link" />
             <child link="${prefix}base_link_inertia" />
-            <!-- 'base_link' is REP-103 aligned (so X+ forward), while the internal
-           frames of the robot/controller have X+ pointing backwards.
-           Use the joint between 'base_link' and 'base_link_inertia' (a dummy
-           link/frame) to introduce the necessary rotation over Z (of pi rad).
-      -->
+            <!--
+                'base_link' is REP-103 aligned (so X+ forward), while the internal
+                frames of the robot/controller have X+ pointing backwards.
+                Use the joint between 'base_link' and 'base_link_inertia' (a dummy
+                link/frame) to introduce the necessary rotation over Z (of pi rad).
+            -->
             <origin xyz="0 0 0" rpy="0 0 ${pi}" />
         </joint>
@@ -278,9 +279,10 @@
         <link name="${prefix}base" />
         <joint name="${prefix}base_link-base_fixed_joint" type="fixed">
-            <!-- Note the rotation over Z of pi radians: as base_link is REP-103
-           aligned (ie: has X+ forward, Y+ left and Z+ up), this is needed
-           to correctly align 'base' with the 'Base' coordinate system of
-           the UR controller.
-      -->
+            <!--
+                Note the rotation over Z of pi radians: as base_link is REP-103
+                aligned (ie: has X+ forward, Y+ left and Z+ up), this is needed
+                to correctly align 'base' with the 'Base' coordinate system of
+                the UR controller.
+            -->
             <origin xyz="0 0 0" rpy="0 0 ${pi}" />
             <parent link="${prefix}base_link" />

Commit message: revert to pure Gazebo installtion

File: catkin_ws/src/rvl_gazebo/xacro/rvl_gazebo.xacro (robot description, xacro)
@@ -94,6 +94,11 @@
         <material>Gazebo/Black</material>
     </gazebo>
-    <xacro:include filename="$(find rvl_gazebo)/xacro/macros/rs_l515_addon.xacro" />
+    <!-- ======================================= REALSENSE ======================================== -->
+    <xacro:include filename="$(find rvl_gazebo)/xacro/macros/rs_l515_addon_rsgz.xacro" />
     <xacro:rs_l515_gazebo_addon camera_name="L515" publish_pointcloud="true"/>
+    <gazebo reference="L515_usb_plug_link">
+        <material>Gazebo/Black</material>
+    </gazebo>
+    <!-- ========================================================================================== -->
     <!--
         Attach the Gazebo model to Gazebo's world frame.

File: catkin_ws/src/rvl_robot_description/xacro/realsense/l515.xacro (robot description, xacro)
@@ -1,8 +1,8 @@
 <?xml version="1.0"?>
 <!--
-License: Apache 2.0. See LICENSE file in root directory.
-Copyright(c) 2017 Intel Corporation. All Rights Reserved
-This is the URDF model for the Intel RealSense L515 camera, in its
-aluminum peripherial evaluation case.
+    License: Apache 2.0. See LICENSE file in root directory.
+    Copyright(c) 2017 Intel Corporation. All Rights Reserved
+    This is the URDF model for the Intel RealSense L515 camera, in its
+    aluminum peripherial evaluation case.
 -->
 <robot name="sensor_l515" xmlns:xacro="http://ros.org/wiki/xacro">
@@ -174,4 +174,5 @@
             </joint>
         </xacro:if>
+        <!-- USB PLUG -->
         <xacro:if value="${add_plug}">
             <xacro:usb_plug parent="${name}_bottom_screw_frame" name="${name}_usb_plug">
