Commit message: weird collision with L515 attached?

File: catkin_ws/src/rvl_gazebo/urdf/rvl_gazebo.urdf (robot description, URDF)
Before this commit: robot rvl_arm_gazebo, 25 links, 24 joints
Links:
- added link L515_bottom_screw_frame
- added link L515_link, mass 0.095; collision cylinder length=0.026 radius=0.0305; visual mesh filename=package://rvl_robot_description/models/realsense/l515.dae
- added link L515_lower_mount
- added link L515_upper_mount
- added link L515_usb_plug_link; collision mesh filename=package://rvl_robot_description/models/realsense/plug_colli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; visual mesh filename=package://rvl_robot_description/models/realsense/plug.stl
Joints:
- added joint L515_joint: type fixed, parent tool0, child L515_bottom_screw_frame, origin xyz=0.0 -0.087 0.0183 rpy=1.5707963267948966 -1.5707963267948966 0.0
- added joint L515_link_joint: type fixed, parent L515_bottom_screw_frame, child L515_link, origin xyz=0.007500000000000001 0.0 0.021150000000000002 rpy=0 0 0
- added joint L515_lower_mount_joint: type fixed, parent L515_bottom_screw_frame, child L515_lower_mount, origin xyz=-0.013999999999999999 0 0.01015 rpy=0 0 0
- added joint L515_upper_mount_joint: type fixed, parent L515_bottom_screw_frame, child L515_upper_mount, origin xyz=-0.013999999999999999 0 0.05015 rpy=0 0 0
- added joint L515_usb_plug_joint: type fixed, parent L515_bottom_screw_frame, child L515_usb_plug_link, origin xyz=-0.0028000000000000004 -0.018 0.018 rpy=0.7853981633974483 0 0 

File: catkin_ws/src/rvl_gazebo/xacro/rvl_gazebo.xacro (robot description, xacro)
@@ -9,4 +9,5 @@
     <xacro:arg name="robotiq_variant" default="2f_85" />
     <xacro:arg name="robotiq_transmission_hw_interface" default="hardware_interface/EffortJointInterface" />
+    <xacro:arg name="realsense_variant" default="l515" />
     <xacro:arg name="safety_limits" default="false" />
     <xacro:arg name="safety_pos_margin" default="0.15" />
@@ -19,4 +20,5 @@
         robotiq_variant="$(arg robotiq_variant)"
         robotiq_transmission_hw_interface="$(arg robotiq_transmission_hw_interface)"
+        realsense_variant="$(arg realsense_variant)"
         safety_limits="$(arg safety_limits)"
         safety_pos_margin="$(arg safety_pos_margin)"

File: catkin_ws/src/rvl_gazebo/xacro/rvl_gazebo_macro.xacro (robot description, xacro)
@@ -7,4 +7,5 @@
         robotiq_variant
         robotiq_transmission_hw_interface:=hardware_interface/EffortJointInterface
+        realsense_variant
         safety_limits:=false
         safety_pos_margin:=0.15
@@ -16,4 +17,5 @@
         <xacro:arg name="robotiq_variant" default="2f_85" />
         <xacro:arg name="robotiq_transmission_hw_interface" default="hardware_interface/EffortJointInterface" />
+        <xacro:arg name="realsense_variant" default="l515" />
         <xacro:arg name="safety_limits" default="false" />
         <xacro:arg name="safety_pos_margin" default="0.15" />
@@ -25,4 +27,5 @@
             robotiq_variant="${robotiq_variant}"
             robotiq_transmission_hw_interface="${robotiq_transmission_hw_interface}"
+            realsense_variant="${realsense_variant}"
             safety_limits="${safety_limits}"
             safety_pos_margin="${safety_pos_margin}"
@@ -156,4 +159,8 @@
             </gazebo>
         </xacro:if>
+        <xacro:if value="${robotiq_variant == '3f'}">
+        </xacro:if>
+        <xacro:if value="${realsense_variant != ''}">
+        </xacro:if>
         <!--
             Inject Gazebo ROS Control plugin, which allows us to use ros_control

File: catkin_ws/src/rvl_robot_description/xacro/custom/mounting_plate.xacro (robot description, xacro)
@@ -18,7 +18,7 @@
             </visual>
             <collision>
-                <origin xyz="0.0 ${0.185/4} ${0.0053/2}" rpy="0.0 0.0 0.0" />
+                <origin xyz="0.0 0.0 0.0" rpy="0.0 0.0 0.0" />
                 <geometry>
-                    <box size="0.075 0.185 0.0053" />
+                    <mesh filename="package://rvl_robot_description/models/mounting_plate.stl" />
                 </geometry>
             </collision>

File: catkin_ws/src/rvl_robot_description/xacro/custom/rvl_arm.xacro (robot description, xacro)
@@ -7,4 +7,5 @@
     <xacro:arg name="robotiq_variant" default="2f_85" />
     <xacro:arg name="robotiq_transmission_hw_interface" default="hardware_interface/EffortJointInterface" />
+    <xacro:arg name="realsense_variant" default="l515" />
     <xacro:arg name="safety_limits" default="false" />
     <xacro:arg name="safety_pos_margin" default="0.15" />
@@ -16,4 +17,5 @@
         robotiq_variant="$(arg robotiq_variant)"
         robotiq_transmission_hw_interface="$(arg robotiq_transmission_hw_interface)"
+        realsense_variant="$(arg realsense_variant)"
         safety_limits="$(arg safety_limits)"
         safety_pos_margin="$(arg safety_pos_margin)"

File: catkin_ws/src/rvl_robot_description/xacro/custom/rvl_ur_robotiq_macro.xacro (robot description, xacro)
@@ -7,26 +7,27 @@
         robotiq_variant
         robotiq_transmission_hw_interface:=hardware_interface/EffortJointInterface
+        realsense_variant
         safety_limits:=false
         safety_pos_margin:=0.15
         safety_k_position:=20">
+        <xacro:property name="tool_rotation" value="${pi/2}" />
         <xacro:property name="coupling_offset" value="0.0053" />
-        <xacro:property name="tool_rotation" value="${pi/2}" />
-        <xacro:property name="camera_placement_offset" value="0.12439" />
-        <xacro:property name="camera_origin_offset" value="0.0061"/>
+        <xacro:property name="plate_offset" value="0.1175" />
+        <!-- TODO: Save dimensions in yaml and load as property -->
+        <xacro:property name="camera_thickness" value="0.061" />
+        <!-- y offset = camera_width / 2 - plate_offset -->
+        <!-- z offset = camera_thickness + mounting_plate_thickness -->
+        <!-- TODO: Make formula adaptive to the rest of RealSense cameras? -->
+        <xacro:property name="camera_placement_xyz" value="0.0 ${camera_thickness/2.0 - plate_offset} ${0.013 + coupling_offset}" />
+        <xacro:property name="camera_placement_rpy" value="${pi/2} ${-pi/2} 0.0" />
         <!-- Universal Robots arm -->
         <xacro:include filename="$(find rvl_robot_description)/xacro/universal_robots/include/ur_macro.xacro" />
-        <xacro:ur_robot
-            prefix="${prefix}"
-            variant="${ur_variant}"
-            transmission_hw_interface="${ur_transmission_hw_interface}"
-            safety_limits="${safety_limits}"
-            safety_pos_margin="${safety_pos_margin}"
-            safety_k_position="${safety_k_position}" />
+        <xacro:ur_robot prefix="${prefix}" variant="${ur_variant}" transmission_hw_interface="${ur_transmission_hw_interface}" safety_limits="${safety_limits}" safety_pos_margin="${safety_pos_margin}" safety_k_position="${safety_k_position}" />
         <!-- Custom L515 mounting plate -->
-        <xacro:include filename="$(find rvl_robot_description)/xacro/custom/mounting_plate.xacro"/>
-        <xacro:L515_mounting_plate prefix="${prefix}"/>
+        <xacro:include filename="$(find rvl_robot_description)/xacro/custom/mounting_plate.xacro" />
+        <xacro:L515_mounting_plate prefix="${prefix}" />
         <joint name="tool0-mounting_plate" type="fixed">
-            <parent link= "${prefix}tool0" />
-            <child link = "${prefix}L515_mounting_plate" />
+            <parent link="${prefix}tool0" />
+            <child link="${prefix}L515_mounting_plate" />
             <origin xyz="0.0 0.0 0.0" rpy="0.0 0.0 ${pi}" />
         </joint>
@@ -34,27 +35,33 @@
         <xacro:if value="${robotiq_variant.startswith('2f')}">
             <xacro:include filename="$(find rvl_robot_description)/xacro/robotiq/include/robotiq_2f_macro.xacro" />
-            <xacro:property name="gripper_height" value="${0.1628 if robotiq_variant[3:] == '85' else 0.2328}" scope="parent"/>
-            <xacro:robotiq_2f_gripper
-                prefix="${prefix}"
-                stroke="${robotiq_variant[3:]}"
-                transmission_hw_interface="${robotiq_transmission_hw_interface}"
-                parent_link="${prefix}tool0"
-                attachment_z="${coupling_offset}"
-                attachment_yaw="${tool_rotation}" />
+            <xacro:property name="gripper_height" value="${0.1628 if robotiq_variant[3:] == '85' else 0.2328}" scope="parent" />
+            <xacro:robotiq_2f_gripper prefix="${prefix}" stroke="${robotiq_variant[3:]}" transmission_hw_interface="${robotiq_transmission_hw_interface}" parent_link="${prefix}tool0" attachment_z="${coupling_offset}" attachment_yaw="${tool_rotation}" />
         </xacro:if>
         <xacro:if value="${robotiq_variant == '3f'}">
             <!-- TODO: Add 3-Finger Robotiq model and xacro -->
         </xacro:if>
-        <!-- Intel RealSense Camera - TBD -->
-        <!-- TODO: Add Intel RealSense L515 (or other variant) support -->
+        <!-- Intel RealSense Camera, only load when needed -->
+        <xacro:if value="${realsense_variant != ''}">
+            <xacro:property name="use_nominal_extrinsics" default="false" />
+            <xacro:property name="add_plug" default="true" />
+            <xacro:property name="use_mesh" default="true" />
+            <!-- RealSense L515 -->
+            <xacro:if value="${realsense_variant == 'l515'}">
+                <xacro:include filename="$(find rvl_robot_description)/xacro/realsense/l515.xacro" />
+                <xacro:sensor_l515 name="L515" parent="${prefix}tool0" use_nominal_extrinsics="${use_nominal_extrinsics}" add_plug="${add_plug}" use_mesh="${use_mesh}">
+                    <origin xyz="${camera_placement_xyz}" rpy="${camera_placement_rpy}" />
+                </xacro:sensor_l515>
+            </xacro:if>
+            <!-- TODO: Add other Intel RealSense camera support -->
+        </xacro:if>
         <!-- Additional link for planning (center of gripper tips when fully closed) -->
         <link name="${prefix}gripper_center_tip" />
         <joint name="${prefix}gripper_center_tip_joint" type="fixed">
-            <parent link="${prefix}tool0"/>
-            <child link="${prefix}gripper_center_tip"/>
-            <origin xyz="0.0 0.0 ${coupling_offset + gripper_height}" rpy="0.0 0.0 0.0"/>
+            <parent link="${prefix}tool0" />
+            <child link="${prefix}gripper_center_tip" />
+            <origin xyz="0.0 0.0 ${coupling_offset + gripper_height}" rpy="0.0 0.0 0.0" />
         </joint>
     </xacro:macro>
     <!-- testing -->
-    <!-- <xacro:rvl_arm prefix="" ur_variant="ur5e" robotiq_variant="2f_85"/> -->
+    <!-- <xacro:rvl_arm prefix="" ur_variant="ur5e" robotiq_variant="2f_85" /> -->
 </robot>
