Commit message: preparing to migrate older UR-Robotiq driver to this repo

File: catkin_ws/src/rvl_robot_description/xacro/realsense/d415.xacro (robot description, xacro)
@@ -8,5 +8,5 @@
 <robot name="sensor_d415" xmlns:xacro="http://ros.org/wiki/xacro">
   <!-- Includes -->
-  <xacro:include filename="$(find rvl_robot_description)/xacro/realsense/materials.xacro" />
+  <xacro:include filename="$(find rvl_robot_description)/xacro/rvl/materials.xacro" />
   <xacro:include filename="$(find rvl_robot_description)/xacro/realsense/usb_plug.xacro" />
   <xacro:macro name="sensor_d415" params="parent *origin  name:=camera  use_nominal_extrinsics:=false add_plug:=false use_mesh:=true">

File: catkin_ws/src/rvl_robot_description/xacro/realsense/d435.xacro (robot description, xacro)
@@ -8,5 +8,5 @@
 <robot name="sensor_d435" xmlns:xacro="http://ros.org/wiki/xacro">
   <!-- Includes -->
-  <xacro:include filename="$(find rvl_robot_description)/xacro/realsense/materials.xacro" />
+  <xacro:include filename="$(find rvl_robot_description)/xacro/rvl/materials.xacro" />
   <xacro:include filename="$(find rvl_robot_description)/xacro/realsense/usb_plug.xacro" />
   <xacro:macro name="sensor_d435" params="parent *origin name:=camera use_nominal_extrinsics:=false add_plug:=false use_mesh:=true">

File: catkin_ws/src/rvl_robot_description/xacro/realsense/d455.xacro (robot description, xacro)
@@ -8,5 +8,5 @@
 <robot name="sensor_d455" xmlns:xacro="http://ros.org/wiki/xacro">
   <!-- Includes -->
-  <xacro:include filename="$(find rvl_robot_description)/xacro/realsense/materials.xacro" />
+  <xacro:include filename="$(find rvl_robot_description)/xacro/rvl/materials.xacro" />
   <xacro:include filename="$(find rvl_robot_description)/xacro/realsense/usb_plug.xacro" />
   <xacro:macro name="sensor_d455" params="parent *origin name:=camera use_nominal_extrinsics:=false">

File: catkin_ws/src/rvl_robot_description/xacro/realsense/l515.xacro (robot description, xacro)
@@ -8,7 +8,7 @@
 <robot name="sensor_l515" xmlns:xacro="http://ros.org/wiki/xacro">
     <!-- Includes -->
-    <xacro:include filename="$(find rvl_robot_description)/xacro/realsense/materials.xacro" />
+    <xacro:include filename="$(find rvl_robot_description)/xacro/rvl/materials.xacro" />
     <xacro:include filename="$(find rvl_robot_description)/xacro/realsense/usb_plug.xacro" /> <!-- this specific plug does not apply to L515 -->
-    <xacro:macro name="sensor_l515" params="parent *origin name:=camera use_nominal_extrinsics:=false add_plug:=false use_mesh:=true">
+    <xacro:macro name="sensor_l515" params="parent *origin name:=camera use_nominal_extrinsics:=false add_plug:=true use_mesh:=true">
         <xacro:property name="M_PI" value="3.1415926535897931" />
         <!--

File: catkin_ws/src/rvl_robot_description/xacro/realsense/r410.xacro (robot description, xacro)
@@ -8,5 +8,5 @@
 <robot name="sensor_r410" xmlns:xacro="http://ros.org/wiki/xacro">
   <!-- Includes -->
-  <xacro:include filename="$(find rvl_robot_description)/xacro/realsense/materials.xacro" />
+  <xacro:include filename="$(find rvl_robot_description)/xacro/rvl/materials.xacro" />
   <xacro:macro name="sensor_r410" params="parent *origin  name:=camera  use_nominal_extrinsics:=false">
     <xacro:property name="M_PI" value="3.1415926535897931" />

File: catkin_ws/src/rvl_robot_description/xacro/realsense/r430.xacro (robot description, xacro)
@@ -8,5 +8,5 @@
 <robot name="sensor_r430" xmlns:xacro="http://ros.org/wiki/xacro">
   <!-- Includes -->
-  <xacro:include filename="$(find rvl_robot_description)/xacro/realsense/materials.xacro" />
+  <xacro:include filename="$(find rvl_robot_description)/xacro/rvl/materials.xacro" />
   <xacro:macro name="sensor_r430" params="parent *origin name:=camera use_nominal_extrinsics:=false">
   <xacro:property name="M_PI" value="3.1415926535897931" />

File: catkin_ws/src/rvl_robot_description/xacro/realsense/realsense_loader.xacro (robot description, xacro)
@@ -3,5 +3,5 @@
     <!-- <xacro:arg name="rs_variant" default="d415"/> -->
     <xacro:arg name="use_nominal_extrinsics" default="false" />
-    <xacro:arg name="add_plug" default="false" />
+    <xacro:arg name="add_plug" default="true" />
     <xacro:arg name="use_mesh" default="true" />
     <!-- needed to make it a property for if statement? -->

File: catkin_ws/src/rvl_robot_description/xacro/robotiq/include/robotiq_2f_common.xacro (robot description, xacro)
@@ -145,6 +145,4 @@
         <xacro:property name="finger_tip_collision_xyz" value="${finger_tip_collision_parameters['origin']['xyz']}" scope="parent" />
         <xacro:property name="finger_tip_collision_rpy" value="${finger_tip_collision_parameters['origin']['rpy']}" scope="parent" />
-        <xacro:property name="finger_tip_collision_material_name" value="${finger_tip_collision_parameters['material']['name']}" scope="parent" />
-        <xacro:property name="finger_tip_collision_material_color" value="${finger_tip_collision_parameters['material']['color']}" scope="parent" />
         <!-- INDIVIDUAL JOINT NAMES -->
         <xacro:property name="knuckle_joint_name" value="${sec_joint_names['base_to_knuckle']}" scope="parent" />

File: catkin_ws/src/rvl_robot_description/xacro/robotiq/include/robotiq_2f_macro.xacro (robot description, xacro)
@@ -134,7 +134,4 @@
                         <box size="${finger_tip_box_dimension}" />
                     </geometry>
-                    <material name="${finger_tip_collision_material_name}">
-                        <color rgba="${finger_tip_collision_material_color}" />
-                    </material>
                 </collision>
             </link>

File: catkin_ws/src/rvl_robot_description/xacro/rvl/multibot.xacro (robot description, xacro)
@@ -1,17 +1,57 @@
 <?xml version="1.0"?>
 <robot xmlns:xacro="http://www.ros.org/wiki/xacro" name="multibot">
+    <!-- ####################################################################### -->
+    <!--                        TWO UNIVERSAL ROBOT UR5e                         -->
+    <!-- ####################################################################### -->
+    <xacro:property name="ur_range" value="0.85" />
+    <xacro:property name="ur_overlap" value="${ur_range * 2.0 - (ur_range * 0.75 * 2.0)}" />
+    <xacro:property name="ur_spacing" value="${0.85 * 2.0 - ur_overlap}" />
     <xacro:include filename="$(find rvl_robot_description)/xacro/universal_robots/include/ur_macro.xacro"/>
-    <xacro:ur_robot prefix="first_" variant="ur5e" />
-    <xacro:ur_robot prefix="second_" variant="ur5e" />
+    <xacro:ur_robot prefix="left_" variant="ur5e" />
+    <xacro:ur_robot prefix="right_" variant="ur5e" />
+    <!-- ####################################################################### -->
+    <!--             TWO ROBOTIQ 2F-85 GRIPPERS ATTACHED TO THE UR5e             -->
+    <!-- ####################################################################### -->
+    <xacro:include filename="$(find rvl_robot_description)/xacro/robotiq/include/robotiq_2f_macro.xacro" />
+    <xacro:robotiq_2f_gripper
+        prefix="left_"
+        stroke="85"
+        transmission_hw_interface="hardware_interface/EffortJointInterface"
+        parent_link="left_tool0"
+        attachment_yaw="${pi/2}" />
+    <xacro:robotiq_2f_gripper
+        prefix="right_"
+        stroke="85"
+        transmission_hw_interface="hardware_interface/EffortJointInterface"
+        parent_link="right_tool0"
+        attachment_yaw="${pi/2}" />
+    <!-- ####################################################################### -->
+    <!--              ADDITIONAL PLANNING JOINT FOR GRIPPER CENTER               -->
+    <!-- ####################################################################### -->
+    <link name="left_gripper_center_tip" />
+    <joint name="left_gripper_center_tip_joint" type="fixed">
+        <parent link="left_tool0" />
+        <child link="left_gripper_center_tip" />
+        <origin xyz="0.0 0.0 ${0.1628 * 0.8}" rpy="0.0 0.0 0.0" />
+    </joint>
+    <link name="right_gripper_center_tip" />
+    <joint name="right_gripper_center_tip_joint" type="fixed">
+        <parent link="right_tool0" />
+        <child link="right_gripper_center_tip" />
+        <origin xyz="0.0 0.0 ${0.1628 * 0.8}" rpy="0.0 0.0 0.0" />
+    </joint>
+    <!-- ####################################################################### -->
+    <!--         MOUNTING THE BOTS TO THE "WORLD" AS A COMMON BASE LINK          -->
+    <!-- ####################################################################### -->
     <link name="world" />
-    <joint name="first_to_platform" type="fixed">
+    <joint name="left_to_world" type="fixed">
         <parent link="world"/>
-        <child link="first_base_link"/>
-        <origin xyz="0 -0.6 0.05"/>
+        <child link="left_base_link"/>
+        <origin xyz="0 0 0" rpy="0 0 ${-pi/2.0}"/>
     </joint>
-    <joint name="second_to_platform" type="fixed">
+    <joint name="right_to_world" type="fixed">
         <parent link="world"/>
-        <child link="second_base_link"/>
-        <origin xyz="0 -1.2 0.05"/>
+        <child link="right_base_link"/>
+        <origin xyz="0 ${ur_spacing} 0" rpy="0 0 ${-pi/2.0}"/>
     </joint>
 </robot>

File: catkin_ws/src/rvl_robot_description/xacro/rvl/rvl_ur.xacro (robot description, xacro)
@@ -28,5 +28,5 @@
     <!-- Intel RealSense L515 -->
     <xacro:include filename="$(find rvl_robot_description)/xacro/realsense/l515.xacro" />
-    <xacro:sensor_l515 name="L515" parent="tool0" add_plug="true">
+    <xacro:sensor_l515 name="L515" parent="tool0">
         <origin xyz="${camera_placement_xyz}" rpy="${camera_placement_rpy}" />
     </xacro:sensor_l515>

File: catkin_ws/src/rvl_robot_description/xacro/universal_robots/include/ur_macro.xacro (robot description, xacro)
@@ -52,5 +52,9 @@
         safety_k_position:=20">
         <!-- Load configuration data from the provided .yaml files -->
-        <xacro:read_model_data joint_limits_parameters_file="$(find rvl_robot_description)/config/universal_robots/${variant}/joint_limits.yaml" kinematics_parameters_file="$(find rvl_robot_description)/config/universal_robots/${variant}/default_kinematics.yaml" physical_parameters_file="$(find rvl_robot_description)/config/universal_robots/${variant}/physical_parameters.yaml" visual_parameters_file="$(find rvl_robot_description)/config/universal_robots/${variant}/visual_parameters.yaml" />
+        <xacro:read_model_data
+            joint_limits_parameters_file="$(find rvl_robot_description)/config/universal_robots/${variant}/joint_limits.yaml"
+            kinematics_parameters_file="$(find rvl_robot_description)/config/universal_robots/${variant}/default_kinematics.yaml"
+            physical_parameters_file="$(find rvl_robot_description)/config/universal_robots/${variant}/physical_parameters.yaml"
+            visual_parameters_file="$(find rvl_robot_description)/config/universal_robots/${variant}/visual_parameters.yaml" />
         <!-- Add URDF transmission elements (for ros_control) -->
         <xacro:ur_arm_transmission prefix="${prefix}" hw_interface="${transmission_hw_interface}" />
