Commit message: updated Fetch collision matrix

File: catkin_ws/src/rvl_robot_description/urdf/rvl_ur10e.urdf (robot description, URDF)
Before this commit: robot rvl_ur, 29 links, 28 joints
Links:
- removed link L515_bottom_screw_frame
- removed link L515_link
- removed link L515_lower_mount
- removed link L515_mounting_plate
- removed link L515_upper_mount
- removed link L515_usb_plug_link
- link base_link_inertia: geometry collision mesh filename=package://rvl_robot_description/models/universal_robots/ur1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; visual mesh filename=package://rvl_robot_description/models/universal_robots/ur1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
- link forearm_link: mass 2.275 -> 3.87; geometry collision mesh filename=package://rvl_robot_description/models/universal_robots/ur1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; visual mesh filename=package://rvl_robot_description/models/universal_robots/ur1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
- link left_bar_link: geometry collision mesh filename=package://rvl_robot_description/models/robotiq/2f_140/colli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 scale=1 1 1; visual mesh filename=package://rvl_robot_description/models/robotiq/2f_140/visua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 scale=1 1 1
- link left_distal_phalanx_link: geometry collision mesh filename=package://rvl_robot_description/models/robotiq/2f_140/colli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 scale=1 1 1; visual mesh filename=package://rvl_robot_description/models/robotiq/2f_140/visua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 scale=1 1 1
- link left_finger_tip_link: geometry collision box size=0.03 0.07 0.0075; visual box size=0.03 0.07 0.0075
- link left_knuckle_link: geometry collision mesh filename=package://rvl_robot_description/models/robotiq/2f_140/colli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 scale=1 1 1; visual mesh filename=package://rvl_robot_description/models/robotiq/2f_140/visua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 scale=1 1 1
- link left_proximal_phalanx_link: geometry collision mesh filename=package://rvl_robot_description/models/robotiq/2f_140/colli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 scale=1 1 1; visual mesh filename=package://rvl_robot_description/models/robotiq/2f_140/visua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 scale=1 1 1
- link right_bar_link: geometry collision mesh filename=package://rvl_robot_description/models/robotiq/2f_140/colli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 scale=1 1 1; visual mesh filename=package://rvl_robot_description/models/robotiq/2f_140/visua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 scale=1 1 1
- link right_distal_phalanx_link: geometry collision mesh filename=package://rvl_robot_description/models/robotiq/2f_140/colli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 scale=1 1 1; visual mesh filename=package://rvl_robot_description/models/robotiq/2f_140/visua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 scale=1 1 1
- link right_finger_tip_link: geometry collision box size=0.03 0.07 0.0075; visual box size=0.03 0.07 0.0075
- link right_knuckle_link: geometry collision mesh filename=package://rvl_robot_description/models/robotiq/2f_140/colli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 scale=1 1 1; visual mesh filename=package://rvl_robot_description/models/robotiq/2f_140/visua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 scale=1 1 1
- link right_proximal_phalanx_link: geometry collision mesh filename=package://rvl_robot_description/models/robotiq/2f_140/colli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 scale=1 1 1; visual mesh filename=package://rvl_robot_description/models/robotiq/2f_140/visua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 scale=1 1 1
- link robotiq_2f_base_palm: geometry collision mesh filename=package://rvl_robot_description/models/robotiq/2f_140/colli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 scale=1 1 1; visual mesh filename=package://rvl_robot_description/models/robotiq/2f_140/visua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 scale=1 1 1
- link shoulder_link: mass 3.7 -> 7.778; geometry collision mesh filename=package://rvl_robot_description/models/universal_robots/ur1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; visual mesh filename=package://rvl_robot_description/models/universal_robots/ur1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
- link upper_arm_link: mass 8.393 -> 12.93; geometry collision mesh filename=package://rvl_robot_description/models/universal_robots/ur1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; visual mesh filename=package://rvl_robot_description/models/universal_robots/ur1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
- link wrist_1_link: mass 1.219 -> 1.96; geometry collision mesh filename=package://rvl_robot_description/models/universal_robots/ur1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; visual mesh filename=package://rvl_robot_description/models/universal_robots/ur1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
- link wrist_2_link: mass 1.219 -> 1.96; geometry collision mesh filename=package://rvl_robot_description/models/universal_robots/ur1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; visual mesh filename=package://rvl_robot_description/models/universal_robots/ur1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
- link wrist_3_link: mass 0.1879 -> 0.202; geometry collision mesh filename=package://rvl_robot_description/models/universal_robots/ur1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; visual mesh filename=package://rvl_robot_description/models/universal_robots/ur1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
Joints:
- removed joint L515_joint
- removed joint L515_link_joint
- removed joint L515_lower_mount_joint
- removed joint L515_upper_mount_joint
- removed joint L515_usb_plug_joint
- removed joint tool0-mounting_plate
- joint elbow_joint: origin xyz=-0.4255477404386134 0 0 rpy=3.141279979860951 3.138418572813499 3.141588694100498 -> xyz=-0.6127 0 0 rpy=0 0 0
- joint gripper_center_tip_joint: origin xyz=0.0 0.0 0.15182 rpy=0.0 0.0 0.0 -> xyz=0.0 0.0 0.14652 rpy=0.0 0.0 0.0
- joint knuckle_joint: axis 1 0 0 -> -1 0 0; limit lower=0.0 upper=0.8 effort=1000 velocity=0.5 -> lower=0 upper=0.7 effort=1000 velocity=0.5; origin xyz=0 -0.0306011 0.054904 rpy=0 0 3.141592654 -> xyz=0 -0.0306011 0.054904 rpy=2.295796327 0 0
- joint left_bar_joint: origin xyz=0 0.0315 -0.0041 rpy=0 0 0 -> xyz=0 0.01821998610742 0.0260018192872234 rpy=0 0 0
- joint left_distal_joint: limit lower=-0.8757 upper=0 effort=1000 velocity=0.5 -> lower=0 upper=0.8757 effort=1000 velocity=0.5; mimic joint=knuckle_joint multiplier=-1 offset=0 -> joint=knuckle_joint multiplier=1 offset=0; origin xyz=0 0.0061 0.0471 rpy=0 0 0 -> xyz=0 0.0817554015893473 -0.0282203446692936 rpy=-0.725 0 0
- joint left_proximal_joint: limit lower=0 upper=0.8757 effort=1000 velocity=0.5 -> lower=-0.8757 upper=0 effort=1000 velocity=0.5; mimic joint=knuckle_joint multiplier=1 offset=0 -> joint=knuckle_joint multiplier=-1 offset=0; origin xyz=0 -0.0127 0.06142 rpy=0 0 3.141592653589793 -> xyz=0 -0.0127 0.06142 rpy=2.2957963267948966 0 0.0
- joint left_tip_joint: origin xyz=0 -0.0220203446692936 0.03242 rpy=0 0 0 -> xyz=0 0.0457554015893473 -0.0272203446692936 rpy=0 0 0
- joint right_bar_joint: origin xyz=0 0.0315 -0.0041 rpy=0 0 0 -> xyz=0 0.01821998610742 0.0260018192872234 rpy=0 0 0
- joint right_distal_joint: limit lower=-0.8757 upper=0 effort=1000 velocity=0.5 -> lower=0 upper=0.8757 effort=1000 velocity=0.5; mimic joint=knuckle_joint multiplier=-1 offset=0 -> joint=knuckle_joint multiplier=1 offset=0; origin xyz=0 0.0061 0.0471 rpy=0 0 0 -> xyz=0 0.0817554015893473 -0.0282203446692936 rpy=-0.725 0 0
- joint right_knuckle_joint: limit lower=0.0 upper=0.8 effort=1000 velocity=0.5 -> lower=-0.725 upper=0 effort=1000 velocity=0.5; mimic joint=knuckle_joint multiplier=1 offset=0 -> joint=knuckle_joint multiplier=-1 offset=0; origin xyz=0 0.0306011 0.054904 rpy=0 0 0 -> xyz=0 0.0306011 0.054904 rpy=2.295796327 0 3.141592654
- joint right_proximal_joint: limit lower=0 upper=0.8757 effort=1000 velocity=0.5 -> lower=-0.8757 upper=0 effort=1000 velocity=0.5; mimic joint=knuckle_joint multiplier=1 offset=0 -> joint=knuckle_joint multiplier=-1 offset=0; origin xyz=0 0.0127 0.06142 rpy=0 0 0.0 -> xyz=0 0.0127 0.06142 rpy=2.2957963267948966 0 -3.141592653589793
- joint right_tip_joint: origin xyz=0 -0.0220203446692936 0.03242 rpy=0 0 0 -> xyz=0 0.0457554015893473 -0.0272203446692936 rpy=0 0 0
- joint shoulder_lift_joint: limit lower=-6.283185307179586 upper=6.283185307179586 effort=150.0 velocity=3.141592653589793 -> lower=-6.283185307179586 upper=6.283185307179586 effort=330.0 velocity=2.0943951023931953; origin xyz=0.0001171864022656332 0 0 rpy=1.568695822980486 0 2.350143582628094e-06 -> xyz=0 0 0 rpy=1.570796327 0 0
- joint shoulder_pan_joint: limit lower=-6.283185307179586 upper=6.283185307179586 effort=150.0 velocity=3.141592653589793 -> lower=-6.283185307179586 upper=6.283185307179586 effort=330.0 velocity=2.0943951023931953; origin xyz=0 0 0.1627616112650263 rpy=0 0 -5.991681506500868e-08 -> xyz=0 0 0.1807 rpy=0 0 0
- joint tool0-robotiq_2f_base_palm: origin xyz=0.0 0.0 0.0053 rpy=0.0 0.0 1.5707963267948966 -> xyz=0.0 0.0 0.0 rpy=0.0 0.0 1.5707963267948966
- joint wrist_1_joint: limit lower=-6.283185307179586 upper=6.283185307179586 effort=28.0 velocity=3.141592653589793 -> lower=-6.283185307179586 upper=6.283185307179586 effort=56.0 velocity=3.141592653589793; origin xyz=-0.3926470322593426 -0.0004490249165745644 0.1335443945419522 rpy=0.003362351718143002 -0.001385386431977988 1.052643010408702e-05 -> xyz=-0.57155 0 0.17415 rpy=0 0 0
- joint wrist_2_joint: limit lower=-6.283185307179586 upper=6.283185307179586 effort=28.0 velocity=3.141592653589793 -> lower=-6.283185307179586 upper=6.283185307179586 effort=56.0 velocity=3.141592653589793; origin xyz=2.411651959975612e-06 -0.09979265928964354 8.42316669864543e-05 rpy=1.569952260231459 0 4.512455664684723e-08 -> xyz=0 -0.11985 -2.458164590756244e-11 rpy=1.570796327 0 0
- joint wrist_3_joint: limit lower=-6.283185307179586 upper=6.283185307179586 effort=28.0 velocity=3.141592653589793 -> lower=-6.283185307179586 upper=6.283185307179586 effort=56.0 velocity=3.141592653589793; origin xyz=-1.62560369067358e-06 0.09963772799936342 0.0001365236554595149 rpy=1.572166526344426 3.141592653589793 -3.14159262258105 -> xyz=0 0.11655 -2.390480459346185e-11 rpy=1.570796326589793 3.141592653589793 3.141592653589793

File: catkin_ws/src/rvl_robot_description/urdf/rvl_ur3e.urdf (robot description, URDF)
Before this commit: robot rvl_ur, 29 links, 28 joints
Links:
- removed link L515_bottom_screw_frame
- removed link L515_link
- removed link L515_lower_mount
- removed link L515_mounting_plate
- removed link L515_upper_mount
- removed link L515_usb_plug_link
- link base_link_inertia: mass 4.0 -> 2.0; geometry collision mesh filename=package://rvl_robot_description/models/universal_robots/ur3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; visual mesh filename=package://rvl_robot_description/models/universal_robots/ur3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
- link forearm_link: mass 2.275 -> 1.26; geometry collision mesh filename=package://rvl_robot_description/models/universal_robots/ur3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; visual mesh filename=package://rvl_robot_description/models/universal_robots/ur3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
- link shoulder_link: mass 3.7 -> 2.0; geometry collision mesh filename=package://rvl_robot_description/models/universal_robots/ur3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; visual mesh filename=package://rvl_robot_description/models/universal_robots/ur3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
- link upper_arm_link: mass 8.393 -> 3.42; geometry collision mesh filename=package://rvl_robot_description/models/universal_robots/ur3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; visual mesh filename=package://rvl_robot_description/models/universal_robots/ur3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
- link wrist_1_link: mass 1.219 -> 0.8; geometry collision mesh filename=package://rvl_robot_description/models/universal_robots/ur3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; visual mesh filename=package://rvl_robot_description/models/universal_robots/ur3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
- link wrist_2_link: mass 1.219 -> 0.8; geometry collision mesh filename=package://rvl_robot_description/models/universal_robots/ur3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; visual mesh filename=package://rvl_robot_description/models/universal_robots/ur3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
- link wrist_3_link: mass 0.1879 -> 0.35; geometry collision mesh filename=package://rvl_robot_description/models/universal_robots/ur3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; visual mesh filename=package://rvl_robot_description/models/universal_robots/ur3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
Joints:
- removed joint L515_joint
- removed joint L515_link_joint
- removed joint L515_lower_mount_joint
- removed joint L515_upper_mount_joint
- removed joint L515_usb_plug_joint
- removed joint tool0-mounting_plate
- joint elbow_joint: limit lower=-3.141592653589793 upper=3.141592653589793 effort=150.0 velocity=3.141592653589793 -> lower=-3.141592653589793 upper=3.141592653589793 effort=28.0 velocity=3.141592653589793; origin xyz=-0.4255477404386134 0 0 rpy=3.141279979860951 3.138418572813499 3.141588694100498 -> xyz=-0.24355 0 0 rpy=0 0 0
- joint gripper_center_tip_joint: origin xyz=0.0 0.0 0.15182 rpy=0.0 0.0 0.0 -> xyz=0.0 0.0 0.14652 rpy=0.0 0.0 0.0
- joint shoulder_lift_joint: limit lower=-6.283185307179586 upper=6.283185307179586 effort=150.0 velocity=3.141592653589793 -> lower=-6.283185307179586 upper=6.283185307179586 effort=56.0 velocity=3.141592653589793; origin xyz=0.0001171864022656332 0 0 rpy=1.568695822980486 0 2.350143582628094e-06 -> xyz=0 0 0 rpy=1.570796327 0 0
- joint shoulder_pan_joint: limit lower=-6.283185307179586 upper=6.283185307179586 effort=150.0 velocity=3.141592653589793 -> lower=-6.283185307179586 upper=6.283185307179586 effort=56.0 velocity=3.141592653589793; origin xyz=0 0 0.1627616112650263 rpy=0 0 -5.991681506500868e-08 -> xyz=0 0 0.15185 rpy=0 0 0
- joint tool0-robotiq_2f_base_palm: origin xyz=0.0 0.0 0.0053 rpy=0.0 0.0 1.5707963267948966 -> xyz=0.0 0.0 0.0 rpy=0.0 0.0 1.5707963267948966
- joint wrist_1_joint: limit lower=-6.283185307179586 upper=6.283185307179586 effort=28.0 velocity=3.141592653589793 -> lower=-6.283185307179586 upper=6.283185307179586 effort=12.0 velocity=6.283185307179586; origin xyz=-0.3926470322593426 -0.0004490249165745644 0.1335443945419522 rpy=0.003362351718143002 -0.001385386431977988 1.052643010408702e-05 -> xyz=-0.2132 0 0.13105 rpy=0 0 0
- joint wrist_2_joint: limit lower=-6.283185307179586 upper=6.283185307179586 effort=28.0 velocity=3.141592653589793 -> lower=-6.283185307179586 upper=6.283185307179586 effort=12.0 velocity=6.283185307179586; origin xyz=2.411651959975612e-06 -0.09979265928964354 8.42316669864543e-05 rpy=1.569952260231459 0 4.512455664684723e-08 -> xyz=0 -0.08535 -1.750557762378351e-11 rpy=1.570796327 0 0
- joint wrist_3_joint: limit lower=-6.283185307179586 upper=6.283185307179586 effort=28.0 velocity=3.141592653589793 -> lower=-6.283185307179586 upper=6.283185307179586 effort=12.0 velocity=6.283185307179586; origin xyz=-1.62560369067358e-06 0.09963772799936342 0.0001365236554595149 rpy=1.572166526344426 3.141592653589793 -3.14159262258105 -> xyz=0 0.0921 -1.8890025766262e-11 rpy=1.570796326589793 3.141592653589793 3.141592653589793

File: catkin_ws/src/rvl_robot_description/xacro/fetch/fetch.urdf (robot description, URDF)
Before this commit: robot fetch, 16 links, 15 joints
Links:
- added link bellows_link2, mass 0.169374038216602; collision mesh filename=package://rvl_robot_description/models/fetch/bellows_link_c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; visual mesh filename=package://rvl_robot_description/models/fetch/bellows_link.S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
- added link estop_link, mass 0.00196130439134723; collision mesh filename=package://rvl_robot_description/models/fetch/estop_link.STL; visual mesh filename=package://rvl_robot_description/models/fetch/estop_link.dae
- added link l_wheel_link, mass 4.3542; collision mesh filename=package://rvl_robot_description/models/fetch/l_wheel_link_c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; visual mesh filename=package://rvl_robot_description/models/fetch/l_wheel_link.S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
- added link r_wheel_link, mass 4.3542; collision mesh filename=package://rvl_robot_description/models/fetch/r_wheel_link_c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; visual mesh filename=package://rvl_robot_description/models/fetch/r_wheel_link.S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
- link fetch_base_link: mass None -> 70.1294
Joints:
- added joint bellows_joint2: type fixed, parent torso_lift_link, child bellows_link2, origin xyz=0 0 0 rpy=0 0 0
- added joint estop_joint: type fixed, parent fetch_base_link, child estop_link, origin xyz=-0.12465 0.23892 0.31127 rpy=1.5708 0 0, axis 0 0 0
- added joint l_wheel_joint: type continuous, parent fetch_base_link, child l_wheel_link, origin xyz=0.0012914 0.18738 0.055325 rpy=-6.123E-17 0 0, axis 0 1 0, limit effort=8.85 velocity=17.4
- added joint r_wheel_joint: type continuous, parent fetch_base_link, child r_wheel_link, origin xyz=0.0012914 -0.18738 0.055325 rpy=-6.123E-17 0 0, axis 0 1 0, limit effort=8.85 velocity=17.4
